Commit message: Your update message

File: src/my_robot_description/urdf/arm.xacro (robot description, xacro)
@@ -45,4 +45,5 @@
         <origin xyz="0 0 ${arm_base_height}" rpy="0 0 0" />
         <axis xyz="0 0 1" />
+        <dynamics damping="0.1" friction="0.2"/>
     </joint>
 </robot>

File: src/my_robot_description/urdf/hruh.xacro (robot description, xacro)
@@ -35,4 +35,5 @@
     <origin xyz="0 0 0.3723" rpy="0 0 0"/>
     <axis xyz="0 0 1"/>
+    <dynamics damping="0.1" friction="0.2"/>
     <limit lower="-1.57" upper="1.57" effort="10" velocity="1.0"/>
   </joint>
@@ -53,4 +54,5 @@
       </geometry>
     </collision>
+    <dynamics damping="0.1" friction="0.2"/>
     <inertial>
       <mass value="0.5"/>
@@ -65,4 +67,5 @@
     <origin xyz="0 0 0" rpy="0 0 0"/>
     <axis xyz="0 0 1"/>
+    <dynamics damping="0.1" friction="0.2"/>
     <limit lower="-1.0" upper="1.0" effort="5" velocity="1.0"/>
   </joint>
@@ -91,4 +94,5 @@
     <origin xyz="0 -0.104 0.315" rpy="0 0 0"/>
     <axis xyz="0 1 0"/>
+    <dynamics damping="0.1" friction="0.2"/>
     <limit lower="-1.57" upper="1.57" effort="10" velocity="1.0"/>
   </joint>
@@ -117,4 +121,5 @@
     <origin xyz="0.01 -0.0795 0.02" rpy="0 0 0"/>
     <axis xyz="1 0 0"/>
+    <dynamics damping="0.1" friction="0.2"/>
     <limit lower="-1.57" upper="0.45" effort="10" velocity="1.0"/>
   </joint>
@@ -221,4 +226,5 @@
     <origin xyz="0 -0.012 0" rpy="0 0 0"/>
     <axis xyz="0 1 0"/>
+    <dynamics damping="0.1" friction="0.2"/>
     <limit lower="0" upper="1.9" effort="10" velocity="1.0"/>
   </joint>
@@ -377,4 +383,5 @@
     <origin xyz="0 0.0015 -0.061" rpy="0 0 0"/>
     <axis xyz="0 0 1"/>
+    <dynamics damping="0.1" friction="0.2"/>
     <limit lower="-1.57" upper="1.57" effort="10" velocity="1.0"/>
   </joint>
@@ -432,4 +439,5 @@
     <origin xyz="-0.021 0 0.018" rpy="0 0 0"/>
     <axis xyz="0 0 1"/>
+    <dynamics damping="0.1" friction="0.2"/>
     <limit lower="-1.8" upper="0" effort="10" velocity="1.0"/>
   </joint>
@@ -458,4 +466,5 @@
     <origin xyz="-0.02 0 0.0017" rpy="0 0 0"/>
     <axis xyz="0 1 0"/>
+    <dynamics damping="0.1" friction="0.2"/>
     <limit lower="-0.9" upper="0" effort="10" velocity="1.0"/>
   </joint>
@@ -484,4 +493,5 @@
     <origin xyz="-0.0259 0 -0.001" rpy="0 0 0"/>
     <axis xyz="0 1 0"/>
+    <dynamics damping="0.1" friction="0.2"/>
     <limit lower="-1.0" upper="0" effort="10" velocity="1.0"/>
   </joint>
@@ -510,4 +520,5 @@
     <origin xyz="-0.0259 0.0015 -0.037" rpy="0 0.18 0"/>
     <axis xyz="1 0 0"/>
+    <dynamics damping="0.1" friction="0.2"/>
     <limit lower="0" upper="1.45" effort="10" velocity="1.0"/>
   </joint>
@@ -536,4 +547,5 @@
     <origin xyz="-0.00 0.00 -0.023" rpy="0 0 0"/>
     <axis xyz="1 0 0"/>
+    <dynamics damping="0.1" friction="0.2"/>
     <limit lower="0" upper="1.20" effort="10" velocity="1.0"/>
     <mimic joint="left_palm_to_finger1_lower" multiplier="1.0" offset="0.0"/>
@@ -563,4 +575,5 @@
     <origin xyz="0.00 0.00 -0.02" rpy="0 0 0"/>
     <axis xyz="1 0 0" rpy="1 0 0"/>
+    <dynamics damping="0.1" friction="0.2"/>
     <limit lower="0" upper="1.20" effort="10" velocity="1.0"/>
     <mimic joint="left_palm_to_finger1_lower" multiplier="1.0" offset="0.0"/>
@@ -590,4 +603,5 @@
     <origin xyz="-0.0058 0.001 -0.039" rpy="0 0 0"/>
     <axis xyz="1 0 0"/>
+    <dynamics damping="0.1" friction="0.2"/>
     <limit lower="0" upper="1.45" effort="10" velocity="1.0"/>
   </joint>
@@ -616,4 +630,5 @@
     <origin xyz="-0.00 0.00 -0.028" rpy="0 0 0"/>
     <axis xyz="1 0 0"/>
+    <dynamics damping="0.1" friction="0.2"/>
     <limit lower="0" upper="1.20" effort="10" velocity="1.0"/>
     <mimic joint="left_palm_to_finger2_lower" multiplier="1.0" offset="0.0"/>
@@ -643,4 +658,5 @@
     <origin xyz="0.00 0.00 -0.026" rpy="0 0 0"/>
     <axis xyz="1 0 0" rpy="1 0 0"/>
+    <dynamics damping="0.1" friction="0.2"/>
     <limit lower="0" upper="1.20" effort="10" velocity="1.0"/>
     <mimic joint="left_palm_to_finger2_lower" multiplier="1.0" offset="0.0"/>
@@ -670,4 +686,5 @@
     <origin xyz="0.013 0.001 -0.0365" rpy="0 -0.195 0"/>
     <axis xyz="1 0 0"/>
+    <dynamics damping="0.1" friction="0.2"/>
     <limit lower="0" upper="1.45" effort="10" velocity="1.0"/>
   </joint>
@@ -696,4 +713,5 @@
     <origin xyz="-0.00 0.00 -0.0255" rpy="0 0 0"/>
     <axis xyz="1 0 0"/>
+    <dynamics damping="0.1" friction="0.2"/>
     <limit lower="0" upper="1.20" effort="10" velocity="1.0"/>
     <mimic joint="left_palm_to_finger3_lower" multiplier="1.0" offset="0.0"/>
@@ -723,4 +741,5 @@
     <origin xyz="0.00 0.00 -0.022" rpy="0 0 0"/>
     <axis xyz="1 0 0" rpy="1 0 0"/>
+    <dynamics damping="0.1" friction="0.2"/>
     <limit lower="0" upper="1.20" effort="10" velocity="1.0"/>
     <mimic joint="left_palm_to_finger3_lower" multiplier="1.0" offset="0.0"/>
@@ -750,4 +769,5 @@
     <origin xyz="0.0273 0.00 -0.0315" rpy="0 -0.379 0"/>
     <axis xyz="1 0 0"/>
+    <dynamics damping="0.1" friction="0.2"/>
     <limit lower="0" upper="1.45" effort="10" velocity="1.0"/>
   </joint>
@@ -776,4 +796,5 @@
     <origin xyz="-0.00 0.00 -0.0185" rpy="0 0 0"/>
     <axis xyz="1 0 0"/>
+    <dynamics damping="0.1" friction="0.2"/>
     <limit lower="0" upper="1.20" effort="10" velocity="1.0"/>
     <mimic joint="left_palm_to_finger4_lower" multiplier="1.0" offset="0.0"/>
@@ -803,4 +824,5 @@
     <origin xyz="0.00 0.00 -0.0155" rpy="0 0 0"/>
     <axis xyz="1 0 0" rpy="1 0 0"/>
+    <dynamics damping="0.1" friction="0.2"/>
     <limit lower="0" upper="1.20" effort="10" velocity="1.0"/>
     <mimic joint="left_palm_to_finger4_lower" multiplier="1.0" offset="0.0"/>
@@ -830,4 +852,5 @@
     <origin xyz="0 0.117 0.315" rpy="0 0 0"/>
     <axis xyz="0 1 0"/>
+    <dynamics damping="0.1" friction="0.2"/>
     <limit lower="-1.57" upper="3.14" effort="10" velocity="1.0"/>
   </joint>
@@ -856,4 +879,5 @@
     <origin xyz="0.0025 0.073 0" rpy="0 0 0"/>
     <axis xyz="1 0 0"/>
+    <dynamics damping="0.1" friction="0.2"/>
     <limit lower="-0.45" upper="1.57" effort="10" velocity="1.0"/>
   </joint>
@@ -960,4 +984,5 @@
     <origin xyz="-0.00159 0.00512 -0.03234 " rpy="0 0 0"/>
     <axis xyz="0 1 0"/>
+    <dynamics damping="0.1" friction="0.2"/>
     <limit lower="0" upper="1.9" effort="10" velocity="1.0"/>
   </joint>
@@ -1116,4 +1141,5 @@
     <origin xyz="0 0 -0.1083" rpy="0 0 0"/>
     <axis xyz="0 0 1"/>
+    <dynamics damping="0.1" friction="0.2"/>
     <limit lower="-1.57" upper="1.57" effort="10" velocity="1.0"/>
   </joint>
@@ -1168,4 +1194,5 @@
     <origin xyz="-0.01443 -0.00369 -0.01635" rpy="0 0 0"/>
     <axis xyz="0 0 1"/>
+    <dynamics damping="0.1" friction="0.2"/>
     <limit lower="0" upper="1.8" effort="10" velocity="1.0"/>
   </joint>
@@ -1194,4 +1221,5 @@
     <origin xyz="-0.0279 0.00204 0" rpy="0 0 0"/>
     <axis xyz="0 1 0"/>
+    <dynamics damping="0.1" friction="0.2"/>
     <limit lower="-0.9" upper="0" effort="10" velocity="1.0"/>
   </joint>
@@ -1220,4 +1248,5 @@
     <origin xyz="-0.0255 0.00034 -0.000915" rpy="0 0 0"/>
     <axis xyz="0 1 0"/>
+    <dynamics damping="0.1" friction="0.2"/>
     <limit lower="-1.0" upper="0" effort="10" velocity="1.0"/>
   </joint>
@@ -1273,4 +1302,5 @@
     <axis xyz="1 0 0"/>
     <limit lower="0" upper="1.20" effort="10" velocity="1.0"/>
+    <dynamics damping="0.1" friction="0.2"/>
     <mimic joint="right_palm_to_finger1_lower" multiplier="1.0" offset="0.0"/>
   </joint>
@@ -1299,4 +1329,5 @@
     <origin xyz="0.00 0.00 -0.02" rpy="0 0 0"/>
     <axis xyz="1 0 0" rpy="1 0 0"/>
+    <dynamics damping="0.1" friction="0.2"/>
     <limit lower="0" upper="1.20" effort="10" velocity="1.0"/>
     <mimic joint="right_palm_to_finger1_lower" multiplier="1.0" offset="0.0"/>
@@ -1326,4 +1357,5 @@
     <origin xyz="-0.0058 -0.0018 -0.072" rpy="0 -0.1 0"/>
     <axis xyz="1 0 0"/>
+    <dynamics damping="0.1" friction="0.2"/>
     <limit lower="-1.45" upper="0" effort="10" velocity="1.0"/>
   </joint>
@@ -1352,4 +1384,5 @@
     <origin xyz="0.00 0.00 -0.02776" rpy="0 0 0"/>
     <axis xyz="1 0 0"/>
+    <dynamics damping="0.1" friction="0.2"/>
     <limit lower="0" upper="1.20" effort="10" velocity="1.0"/>
     <mimic joint="right_palm_to_finger2_lower" multiplier="1.0" offset="0.0"/>
@@ -1379,4 +1412,5 @@
     <origin xyz="0.00 0.00 -0.02388" rpy="0 0 0"/>
     <axis xyz="1 0 0" rpy="1 0 0"/>
+    <dynamics damping="0.1" friction="0.2"/>
     <limit lower="0" upper="1.20" effort="10" velocity="1.0"/>
     <mimic joint="right_palm_to_finger2_lower" multiplier="1.0" offset="0.0"/>
@@ -1406,4 +1440,5 @@
     <origin xyz="0.0125 -0.0021 -0.068" rpy="0 -0.27 0"/>
     <axis xyz="1 0 0"/>
+    <dynamics damping="0.1" friction="0.2"/>
     <limit lower="-1.45" upper="0" effort="10" velocity="1.0"/>
   </joint>
@@ -1432,4 +1467,5 @@
     <origin xyz="0.00 0.00 -0.02493 " rpy="0 0 0"/>
     <axis xyz="1 0 0"/>
+    <dynamics damping="0.1" friction="0.2"/>
     <limit lower="0" upper="1.20" effort="10" velocity="1.0"/>
     <mimic joint="right_palm_to_finger3_lower" multiplier="1.0" offset="0.0"/>
@@ -1459,4 +1495,5 @@
     <origin xyz="0.00 0.00 -0.02178" rpy="0 0 0"/>
     <axis xyz="1 0 0" rpy="1 0 0"/>
+    <dynamics damping="0.1" friction="0.2"/>
     <limit lower="0" upper="1.20" effort="10" velocity="1.0"/>
     <mimic joint="right_palm_to_finger3_lower" multiplier="1.0" offset="0.0"/>
@@ -1486,4 +1523,5 @@
     <origin xyz="0.0273 -0.0021 -0.0620" rpy="0 -0.45 0"/>
     <axis xyz="1 0 0"/>
+    <dynamics damping="0.1" friction="0.2"/>
     <limit lower="-1.45" upper="0" effort="10" velocity="1.0"/>
   </joint>
@@ -1512,4 +1550,5 @@
     <origin xyz="0.00 0.00 -0.01822 " rpy="0 0 0"/>
     <axis xyz="1 0 0"/>
+    <dynamics damping="0.1" friction="0.2"/>
     <limit lower="0" upper="1.20" effort="10" velocity="1.0"/>
     <mimic joint="right_palm_to_finger4_lower" multiplier="1.0" offset="0.0"/>
@@ -1539,4 +1578,5 @@
     <origin xyz="0.00 0.00 -0.01509" rpy="0 0 0"/>
     <axis xyz="1 0 0" rpy="1 0 0"/>
+    <dynamics damping="0.1" friction="0.2"/>
     <limit lower="0" upper="1.20" effort="10" velocity="1.0"/>
     <mimic joint="right_palm_to_finger4_lower" multiplier="1.0" offset="0.0"/>
@@ -1566,13 +1606,12 @@
   </gazebo> -->
   <ros2_control name="GazeboSystem" type="system">
-  <!-- <hardware>
-    <plugin>gazebo_ros2_control/GazeboSystem</plugin>
-  </hardware> -->
-  <joint name="left_palm_to_finger1_lower">
-    <command_interface name="position"/>
-    <state_interface name="position"/>
-    <state_interface name="velocity"/>
-  </joint>
-  <!-- Add similar blocks for each actuated joint -->
+    <hardware>
+      <plugin>gazebo_ros2_control/GazeboSystem</plugin>
+    </hardware>
+    <joint name="right_shoulder_to_bisecp">
+      <command_interface name="position"/>
+      <state_interface name="position"/>
+    </joint>
+    <!-- Repeat for all other joints -->
   </ros2_control>
 </robot>

File: src/my_robot_description/urdf/my_robot.urdf.xacro (robot description, xacro)
@@ -12,9 +12,4 @@
         <origin xyz="${base_length / 10.0} 0 ${base_height}" rpy="0 0 3.14" />
     </joint>
-    <!-- <joint name="arm_chest_joint" type="fixed">
-        <parent link="forearm_link" />
-        <child link="chest_hruh" />
-        <origin xyz="${base_length / 50.0} 0 ${-forearm_length/4}" rpy="0 0 0" />
-    </joint> -->
     <gazebo>
         <plugin name="gazebo_ros2_control" filename="libgazebo_ros2_control.so">
