Commit message: Your update message

File: src/my_robot_description/urdf/arm_gazebo.xacro (robot description, xacro)
@@ -26,3 +26,10 @@
         </plugin>
     </gazebo>
+    <gazebo>
+        <plugin
+            filename="gz-sim-joint-state-publisher-system"
+            name="gz::sim::systems::JointStatePublisher">
+            <joint_name>mobile_base_arm_joint</joint_name>
+        </plugin>
+    </gazebo>
 </robot>

File: src/my_robot_description/urdf/hruh.xacro (robot description, xacro)
@@ -27,4 +27,9 @@
   </joint>
   <gazebo reference="chest_hruh">
+      <selfCollide>true</selfCollide>
+  </gazebo>
+  <gazebo reference="chest_hruh">
+      <mu>1.1</mu>
+      <mu2>1.1</mu2>
       <material>Gazebo/Wood</material>
   </gazebo>
@@ -61,4 +66,7 @@
     </inertial>
   </link>
+  <gazebo reference="neck">
+      <selfCollide>true</selfCollide>
+  </gazebo>
   <!-- Head -->
   <joint name="neck_to_head" type="revolute">
@@ -68,5 +76,5 @@
     <axis xyz="0 0 1"/>
     <dynamics damping="1" friction="2"/>
-    <limit lower="-1.0" upper="1.0" effort="5" velocity="1.0"/>
+    <limit lower="-1.0" upper="1.0" effort="500" velocity="1.0"/>
   </joint>
   <link name="head_base">
@@ -88,4 +96,7 @@
     </inertial>
   </link>
+  <gazebo reference="head_base">
+      <selfCollide>true</selfCollide>
+  </gazebo>
   <!-- Left Shoulder Joint -->
   <joint name="chest_to_left_shoulder" type="revolute">
@@ -115,4 +126,7 @@
     </inertial>
   </link>
+  <gazebo reference="left_shoulder">
+      <selfCollide>true</selfCollide>
+  </gazebo>
   <!-- Left S to bisecp Arm Joint -->
   <joint name="left_shoulder_to_bisecp" type="revolute">
@@ -142,4 +156,7 @@
     </inertial>
   </link>
+  <gazebo reference="left_S_to_Bisecp">
+      <selfCollide>true</selfCollide>
+  </gazebo>
   <!-- Left Bisecp uper Joint -->
   <joint name="left_S_to_bisecp_upper" type="fixed">
@@ -168,4 +185,7 @@
     </inertial>
   </link>
+  <gazebo reference="left_bisecp_upper">
+      <selfCollide>true</selfCollide>
+  </gazebo>
   <!-- Left Bisecp lower Joint -->
   <joint name="left_bisecp_uper_to_lower" type="fixed">
@@ -194,10 +214,14 @@
     </inertial>
   </link>
-<!-- Left elbow inword Joint -->
-  <joint name="left_bisecp_to_elbow_inword" type="fixed">
+  <gazebo reference="left_bisecp_lower">
+      <selfCollide>true</selfCollide>
+  </gazebo>
+  <!-- Left elbow inword Joint -->
+  <joint name="left_bisecp_to_elbow_inword" type="revolute">
     <parent link="left_bisecp_lower"/>
     <child link="left_elbow_inword"/>
     <origin xyz="0. 0 -0.12" rpy="0 0 0"/>
-    <axis xyz="0 0 0"/>
+    <axis xyz="0 0 1"/>
+    <dynamics damping="1" friction="2"/>
     <limit lower="-1.57" upper="1.57" effort="500" velocity="1.0"/>
   </joint>
@@ -220,4 +244,7 @@
     </inertial>
   </link>
+  <gazebo reference="left_elbow_inword">
+      <selfCollide>true</selfCollide>
+  </gazebo>
   <!-- Left elbow midle Joint -->
   <joint name="left_elbow_inword_to_midle" type="revolute">
@@ -247,4 +274,7 @@
     </inertial>
   </link>
+  <gazebo reference="left_elbow_midle">
+      <selfCollide>true</selfCollide>
+  </gazebo>
   <!-- Left elbow outword Joint -->
   <joint name="left_elbow_midle_to_outword" type="fixed">
@@ -273,4 +303,7 @@
     </inertial>
   </link>
+  <gazebo reference="left_elbow_outword">
+      <selfCollide>true</selfCollide>
+  </gazebo>
   <!-- Left elbow to forarm upper Joint -->
   <joint name="left_elbow_midle_forarm_upper" type="fixed">
@@ -299,4 +332,7 @@
     </inertial>
   </link>
+  <gazebo reference="left_elbow_to_forarm_upper">
+      <selfCollide>true</selfCollide>
+  </gazebo>
   <!-- Left forarm upper to lower Joint -->
   <joint name="left_forarm_upper_to_lower_1" type="fixed">
@@ -325,4 +361,7 @@
     </inertial>
   </link>
+  <gazebo reference="left_forarm_lower_1">
+      <selfCollide>true</selfCollide>
+  </gazebo>
   <!-- Left forarm internal support -->
   <joint name="left_forarm_lower_1_to_internal_support" type="fixed">
@@ -351,4 +390,7 @@
     </inertial>
   </link>
+  <gazebo reference="left_forarm_internal_support">
+      <selfCollide>true</selfCollide>
+  </gazebo>
   <!-- Left forarm cover joint -->
   <joint name="left_internal_support_to_cover" type="fixed">
@@ -377,4 +419,7 @@
     </inertial>
   </link>
+  <gazebo reference="left_forarm_cover">
+      <selfCollide>true</selfCollide>
+  </gazebo>
   <!-- Left bisecp to wrist Joint -->
   <joint name="left_forarm_to_wrist" type="revolute">
@@ -407,4 +452,7 @@
       <material>Gazebo/Orange</material>
   </gazebo>
+  <gazebo reference="left_wrist">
+      <material>Gazebo/Orange</material>
+  </gazebo>
   <!-- Left palm joint -->
   <joint name="left_wrist_to_palm" type="fixed">
@@ -433,4 +481,7 @@
     </inertial>
   </link>
+  <gazebo reference="left_palm">
+      <selfCollide>true</selfCollide>
+  </gazebo>
   <!-- Left palm to thomb joint -->
   <joint name="left_palm_to_thomb" type="revolute">
@@ -953,9 +1004,10 @@
   </link>
   <!-- Right elbow inword Joint -->
-  <joint name="right_bisecp_to_elbow_inword" type="fixed">
+  <joint name="right_bisecp_to_elbow_inword" type="revolute">
     <parent link="right_bisecp_lower"/>
     <child link="right_elbow_inword"/>
     <origin xyz="0. 0 -0.0873" rpy="0 0 0"/>
-    <axis xyz="0 0 0"/>
+    <axis xyz="0 0 1"/>
+    <dynamics damping="1" friction="2"/>
     <limit lower="-1.57" upper="1.57" effort="500" velocity="1.0"/>
   </joint>
@@ -1274,6 +1326,7 @@
     <child link="right_finger1_lower"/>
     <origin xyz="-0.0249 -0.00225 -0.0708" rpy="0 0.18 0"/>
-    <axis xyz="1 0 0"/>
-    <limit lower="-1.45" upper="0" effort="500" velocity="1.0"/>
+    <axis xyz="-1 0 0"/>
+    <dynamics damping="1" friction="2"/>
+    <limit lower="0" upper="1.45" effort="500" velocity="1.0"/>
   </joint>
   <link name="right_finger1_lower">
@@ -1300,5 +1353,5 @@
     <child link="right_finger1_middle"/>
     <origin xyz="0.00 0.00 -0.023" rpy="0 0 0"/>
-    <axis xyz="1 0 0"/>
+    <axis xyz="-1 0 0"/>
     <limit lower="0" upper="1.20" effort="500" velocity="1.0"/>
     <dynamics damping="1" friction="2"/>
@@ -1328,5 +1381,5 @@
     <child link="right_finger1_upper"/>
     <origin xyz="0.00 0.00 -0.02" rpy="0 0 0"/>
-    <axis xyz="1 0 0" rpy="1 0 0"/>
+    <axis xyz="-1 0 0" rpy="1 0 0"/>
     <dynamics damping="1" friction="2"/>
     <limit lower="0" upper="1.20" effort="500" velocity="1.0"/>
@@ -1356,7 +1409,7 @@
     <child link="right_finger2_lower"/>
     <origin xyz="-0.0058 -0.0018 -0.072" rpy="0 -0.1 0"/>
-    <axis xyz="1 0 0"/>
-    <dynamics damping="1" friction="2"/>
-    <limit lower="-1.45" upper="0" effort="500" velocity="1.0"/>
+    <axis xyz="-1 0 0"/>
+    <dynamics damping="1" friction="2"/>
+    <limit lower="0" upper="1.45" effort="500" velocity="1.0"/>
   </joint>
   <link name="right_finger2_lower">
@@ -1383,5 +1436,5 @@
     <child link="right_finger2_middle"/>
     <origin xyz="0.00 0.00 -0.02776" rpy="0 0 0"/>
-    <axis xyz="1 0 0"/>
+    <axis xyz="-1 0 0"/>
     <dynamics damping="1" friction="2"/>
     <limit lower="0" upper="1.20" effort="500" velocity="1.0"/>
@@ -1411,5 +1464,5 @@
     <child link="right_finger2_upper"/>
     <origin xyz="0.00 0.00 -0.02388" rpy="0 0 0"/>
-    <axis xyz="1 0 0" rpy="1 0 0"/>
+    <axis xyz="-1 0 0" rpy="1 0 0"/>
     <dynamics damping="1" friction="2"/>
     <limit lower="0" upper="1.20" effort="500" velocity="1.0"/>
@@ -1439,7 +1492,7 @@
     <child link="right_finger3_lower"/>
     <origin xyz="0.0125 -0.0021 -0.068" rpy="0 -0.27 0"/>
-    <axis xyz="1 0 0"/>
-    <dynamics damping="1" friction="2"/>
-    <limit lower="-1.45" upper="0" effort="500" velocity="1.0"/>
+    <axis xyz="-1 0 0"/>
+    <dynamics damping="1" friction="2"/>
+    <limit lower="0" upper="1.45" effort="500" velocity="1.0"/>
   </joint>
   <link name="right_finger3_lower">
@@ -1466,5 +1519,5 @@
     <child link="right_finger3_middle"/>
     <origin xyz="0.00 0.00 -0.02493 " rpy="0 0 0"/>
-    <axis xyz="1 0 0"/>
+    <axis xyz="-1 0 0"/>
     <dynamics damping="1" friction="2"/>
     <limit lower="0" upper="1.20" effort="500" velocity="1.0"/>
@@ -1494,5 +1547,5 @@
     <child link="right_finger3_upper"/>
     <origin xyz="0.00 0.00 -0.02178" rpy="0 0 0"/>
-    <axis xyz="1 0 0" rpy="1 0 0"/>
+    <axis xyz="-1 0 0" rpy="1 0 0"/>
     <dynamics damping="1" friction="2"/>
     <limit lower="0" upper="1.20" effort="500" velocity="1.0"/>
@@ -1522,7 +1575,7 @@
     <child link="right_finger4_lower"/>
     <origin xyz="0.0273 -0.0021 -0.0620" rpy="0 -0.45 0"/>
-    <axis xyz="1 0 0"/>
-    <dynamics damping="1" friction="2"/>
-    <limit lower="-1.45" upper="0" effort="500" velocity="1.0"/>
+    <axis xyz="-1 0 0"/>
+    <dynamics damping="1" friction="2"/>
+    <limit lower="0" upper="1.45" effort="500" velocity="1.0"/>
   </joint>
   <link name="right_finger4_lower">
@@ -1549,5 +1602,5 @@
     <child link="right_finger4_middle"/>
     <origin xyz="0.00 0.00 -0.01822 " rpy="0 0 0"/>
-    <axis xyz="1 0 0"/>
+    <axis xyz="-1 0 0"/>
     <dynamics damping="1" friction="2"/>
     <limit lower="0" upper="1.20" effort="500" velocity="1.0"/>
@@ -1577,5 +1630,5 @@
     <child link="right_finger4_upper"/>
     <origin xyz="0.00 0.00 -0.01509" rpy="0 0 0"/>
-    <axis xyz="1 0 0" rpy="1 0 0"/>
+    <axis xyz="-1 0 0" rpy="1 0 0"/>
     <dynamics damping="1" friction="2"/>
     <limit lower="0" upper="1.20" effort="500" velocity="1.0"/>

File: src/my_robot_description/urdf/hruh_gazebo.xacro (robot description, xacro)
@@ -20,4 +20,11 @@
       <i_min>-6</i_min><i_max>6</i_max>
     </plugin>
+     <!-- left_bisecp_to_elbow_inword -->
+    <plugin filename="gz-sim-joint-position-controller-system"
+        name="gz::sim::systems::JointPositionController">
+      <joint_name>left_bisecp_to_elbow_inword</joint_name>
+      <p_gain>300</p_gain><i_gain>2</i_gain><d_gain>3</d_gain>
+      <i_min>-6</i_min><i_max>6</i_max>
+    </plugin>
     <!-- left_elbow_inword_to_midle -->
     <plugin filename="gz-sim-joint-position-controller-system"
@@ -100,4 +107,11 @@
       <i_min>-6</i_min><i_max>6</i_max>
     </plugin>
+    <!-- right_bisecp_to_elbow_inword -->
+    <plugin filename="gz-sim-joint-position-controller-system"
+        name="gz::sim::systems::JointPositionController">
+      <joint_name>right_bisecp_to_elbow_inword</joint_name>
+      <p_gain>300</p_gain><i_gain>2</i_gain><d_gain>3</d_gain>
+      <i_min>-6</i_min><i_max>6</i_max>
+    </plugin>
     <!-- right_elbow_inword_to_midle -->
     <plugin filename="gz-sim-joint-position-controller-system"
@@ -173,3 +187,21 @@
     </plugin>
   </gazebo>
+  <!-- chest to neck -->
+  <gazebo>
+    <plugin filename="gz-sim-joint-position-controller-system"
+            name="gz::sim::systems::JointPositionController">
+      <joint_name>chest_to_neck</joint_name>
+      <p_gain>300</p_gain><i_gain>2</i_gain><d_gain>3</d_gain>
+      <i_min>-6</i_min><i_max>6</i_max>
+    </plugin>
+  </gazebo>
+  <!-- neck to head -->
+  <gazebo>
+    <plugin filename="gz-sim-joint-position-controller-system"
+            name="gz::sim::systems::JointPositionController">
+      <joint_name>neck_to_head</joint_name>
+      <p_gain>300</p_gain><i_gain>2</i_gain><d_gain>3</d_gain>
+      <i_min>-6</i_min><i_max>6</i_max>
+    </plugin>
+  </gazebo>
 </robot>

File: src/my_robot_description/urdf/my_robot.urdf.xacro (robot description, xacro)
@@ -16,21 +16,5 @@
     </joint>
     <gazebo>
-        <plugin
-            filename="gz-sim-joint-state-publisher-system"
-            name="gz::sim::systems::JointStatePublisher">
-            <joint_name>mobile_base_arm_joint</joint_name>
-        </plugin>
+        <selfCollide>true</selfCollide>
     </gazebo>
-    <!-- <gazebo>
-        <plugin filename="libgz_ros2_control-system.so"
-                name="gz_ros2_control::GazeboSimROS2ControlPlugin">
-                <parameters>$(find my_robot_description)/config/ros2_controllers.yaml</parameters>
-        </plugin>
-    </gazebo> -->
-    <!-- <gazebo>
-        <plugin name="gazebo_ros2_control" filename="libgazebo_ros2_control.so">
-            <robot_param>robot_description</robot_param>
-            <parameters>$(find my_robot_description)/config/controllers.yaml</parameters>
-        </plugin>
-    </gazebo> -->
 </robot>
