Commit message: Your update message

File: src/my_robot_description/urdf/hruh.xacro (robot description, xacro)
@@ -5,5 +5,5 @@
     <visual>
       <geometry>
-        <mesh filename="package://my_robot_description/meshes/chest/chest.STL" scale="1 1 1"/>
+        <mesh filename="file:///home/shreyas/ros2_ws/src/my_robot_description/meshes/chest/chest.STL" scale="1 1 1"/>
       </geometry>
       <material name="grey" />
@@ -12,5 +12,5 @@
     <collision>
       <geometry>
-        <mesh filename="package://my_robot_description/meshes/chest/chest.STL" scale="1 1 1"/>
+        <mesh filename="file:///home/shreyas/ros2_ws/src/my_robot_description/meshes/chest/chest.STL" scale="1 1 1"/>
       </geometry>
     </collision>
@@ -41,5 +41,5 @@
       <origin xyz="0 0 0" rpy="0 0 0"/>
       <geometry>
-        <mesh filename="package://my_robot_description/meshes/neck/neck.STL" scale="1 1 1"/>
+        <mesh filename="file:///home/shreyas/ros2_ws/src/my_robot_description/meshes/neck/neck.STL" scale="1 1 1"/>
       </geometry>
       <material name="" >
@@ -50,5 +50,5 @@
       <origin xyz="0 0 0" rpy="0 0 0"/>
       <geometry>
-        <mesh filename="package://my_robot_description/meshes/neck/neck.STL" scale="1 1 1"/>
+        <mesh filename="file:///home/shreyas/ros2_ws/src/my_robot_description/meshes/neck/neck.STL" scale="1 1 1"/>
       </geometry>
     </collision>
@@ -70,11 +70,11 @@
     <visual>
       <geometry>
-        <mesh filename="package://my_robot_description/meshes/head/head.stl" scale="1 1 1"/>
-      </geometry>
-      <material name="grey" />
-    </visual>
-    <collision>
-      <geometry>
-      <mesh filename="package://my_robot_description/meshes/head/head.stl" scale="1 1 1"/>
+        <mesh filename="file:///home/shreyas/ros2_ws/src/my_robot_description/meshes/head/head.stl" scale="1 1 1"/>
+      </geometry>
+      <material name="grey" />
+    </visual>
+    <collision>
+      <geometry>
+      <mesh filename="file:///home/shreyas/ros2_ws/src/my_robot_description/meshes/head/head.stl" scale="1 1 1"/>
       </geometry>
     </collision>
@@ -96,11 +96,11 @@
     <visual>
       <geometry>
-        <mesh filename="package://my_robot_description/meshes/left_arm/left_S_to_C.stl" scale="0.15 0.15 0.15"/>
-      </geometry>
-      <material name="grey" />
-    </visual>
-    <collision>
-      <geometry>
-        <mesh filename="package://my_robot_description/meshes/left_arm/left_S_to_C.stl" scale="0.15 0.15 0.15"/>
+        <mesh filename="file:///home/shreyas/ros2_ws/src/my_robot_description/meshes/left_arm/left_S_to_C.stl" scale="0.15 0.15 0.15"/>
+      </geometry>
+      <material name="grey" />
+    </visual>
+    <collision>
+      <geometry>
+        <mesh filename="file:///home/shreyas/ros2_ws/src/my_robot_description/meshes/left_arm/left_S_to_C.stl" scale="0.15 0.15 0.15"/>
       </geometry>
     </collision>
@@ -122,11 +122,11 @@
     <visual>
       <geometry>
-        <mesh filename="package://my_robot_description/meshes/left_arm/left_S_to_Bisecp.stl" scale="0.15 0.15 0.15"/>
-      </geometry>
-      <material name="grey" />
-    </visual>
-    <collision>
-      <geometry>
-        <mesh filename="package://my_robot_description/meshes/left_arm/left_S_to_Bisecp.stl" scale="0.15 0.15 0.15"/>
+        <mesh filename="file:///home/shreyas/ros2_ws/src/my_robot_description/meshes/left_arm/left_S_to_Bisecp.stl" scale="0.15 0.15 0.15"/>
+      </geometry>
+      <material name="grey" />
+    </visual>
+    <collision>
+      <geometry>
+        <mesh filename="file:///home/shreyas/ros2_ws/src/my_robot_description/meshes/left_arm/left_S_to_Bisecp.stl" scale="0.15 0.15 0.15"/>
       </geometry>
     </collision>
@@ -148,11 +148,11 @@
     <visual>
       <geometry>
-        <mesh filename="package://my_robot_description/meshes/left_arm/Left_bisecp_uper.stl" scale="0.15 0.15 0.15"/>
-      </geometry>
-      <material name="grey" />
-    </visual>
-    <collision>
-      <geometry>
-        <mesh filename="package://my_robot_description/meshes/left_arm/Left_bisecp_uper.stl" scale="0.15 0.15 0.15"/>
+        <mesh filename="file:///home/shreyas/ros2_ws/src/my_robot_description/meshes/left_arm/Left_bisecp_uper.stl" scale="0.15 0.15 0.15"/>
+      </geometry>
+      <material name="grey" />
+    </visual>
+    <collision>
+      <geometry>
+        <mesh filename="file:///home/shreyas/ros2_ws/src/my_robot_description/meshes/left_arm/Left_bisecp_uper.stl" scale="0.15 0.15 0.15"/>
       </geometry>
     </collision>
@@ -174,11 +174,11 @@
     <visual>
       <geometry>
-        <mesh filename="package://my_robot_description/meshes/left_arm/left_Bisecp_lower.stl" scale="0.15 0.15 0.15"/>
-      </geometry>
-      <material name="grey" />
-    </visual>
-    <collision>
-      <geometry>
-        <mesh filename="package://my_robot_description/meshes/left_arm/left_Bisecp_lower.stl" scale="0.15 0.15 0.15"/>
+        <mesh filename="file:///home/shreyas/ros2_ws/src/my_robot_description/meshes/left_arm/left_Bisecp_lower.stl" scale="0.15 0.15 0.15"/>
+      </geometry>
+      <material name="grey" />
+    </visual>
+    <collision>
+      <geometry>
+        <mesh filename="file:///home/shreyas/ros2_ws/src/my_robot_description/meshes/left_arm/left_Bisecp_lower.stl" scale="0.15 0.15 0.15"/>
       </geometry>
     </collision>
@@ -200,11 +200,11 @@
     <visual>
       <geometry>
-        <mesh filename="package://my_robot_description/meshes/left_arm/left_elbow_inword.stl" scale="0.15 0.15 0.15"/>
-      </geometry>
-      <material name="grey" />
-    </visual>
-    <collision>
-      <geometry>
-        <mesh filename="package://my_robot_description/meshes/left_arm/left_elbow_inword.stl" scale="0.15 0.15 0.15"/>
+        <mesh filename="file:///home/shreyas/ros2_ws/src/my_robot_description/meshes/left_arm/left_elbow_inword.stl" scale="0.15 0.15 0.15"/>
+      </geometry>
+      <material name="grey" />
+    </visual>
+    <collision>
+      <geometry>
+        <mesh filename="file:///home/shreyas/ros2_ws/src/my_robot_description/meshes/left_arm/left_elbow_inword.stl" scale="0.15 0.15 0.15"/>
       </geometry>
     </collision>
@@ -226,11 +226,11 @@
     <visual>
       <geometry>
-        <mesh filename="package://my_robot_description/meshes/left_arm/left_elbow_midle.stl" scale="0.15 0.15 0.15"/>
-      </geometry>
-      <material name="grey" />
-    </visual>
-    <collision>
-      <geometry>
-        <mesh filename="package://my_robot_description/meshes/left_arm/left_elbow_midle.stl" scale="0.15 0.15 0.15"/>
+        <mesh filename="file:///home/shreyas/ros2_ws/src/my_robot_description/meshes/left_arm/left_elbow_midle.stl" scale="0.15 0.15 0.15"/>
+      </geometry>
+      <material name="grey" />
+    </visual>
+    <collision>
+      <geometry>
+        <mesh filename="file:///home/shreyas/ros2_ws/src/my_robot_description/meshes/left_arm/left_elbow_midle.stl" scale="0.15 0.15 0.15"/>
       </geometry>
     </collision>
@@ -252,11 +252,11 @@
     <visual>
       <geometry>
-        <mesh filename="package://my_robot_description/meshes/left_arm/Left_elbow_outword.stl" scale="0.15 0.15 0.15"/>
-      </geometry>
-      <material name="grey" />
-    </visual>
-    <collision>
-      <geometry>
-        <mesh filename="package://my_robot_description/meshes/left_arm/Left_elbow_outword.stl" scale="0.15 0.15 0.15"/>
+        <mesh filename="file:///home/shreyas/ros2_ws/src/my_robot_description/meshes/left_arm/Left_elbow_outword.stl" scale="0.15 0.15 0.15"/>
+      </geometry>
+      <material name="grey" />
+    </visual>
+    <collision>
+      <geometry>
+        <mesh filename="file:///home/shreyas/ros2_ws/src/my_robot_description/meshes/left_arm/Left_elbow_outword.stl" scale="0.15 0.15 0.15"/>
       </geometry>
     </collision>
@@ -278,11 +278,11 @@
     <visual>
       <geometry>
-        <mesh filename="package://my_robot_description/meshes/left_arm/left_elbow_to_forarm_upper.stl" scale="0.15 0.15 0.15"/>
-      </geometry>
-      <material name="grey" />
-    </visual>
-    <collision>
-      <geometry>
-        <mesh filename="package://my_robot_description/meshes/left_arm/left_elbow_to_forarm_upper.stl" scale="0.15 0.15 0.15"/>
+        <mesh filename="file:///home/shreyas/ros2_ws/src/my_robot_description/meshes/left_arm/left_elbow_to_forarm_upper.stl" scale="0.15 0.15 0.15"/>
+      </geometry>
+      <material name="grey" />
+    </visual>
+    <collision>
+      <geometry>
+        <mesh filename="file:///home/shreyas/ros2_ws/src/my_robot_description/meshes/left_arm/left_elbow_to_forarm_upper.stl" scale="0.15 0.15 0.15"/>
       </geometry>
     </collision>
@@ -304,11 +304,11 @@
     <visual>
       <geometry>
-        <mesh filename="package://my_robot_description/meshes/left_arm/Left_forarm_lower_1.stl" scale="0.15 0.15 0.15"/>
-      </geometry>
-      <material name="grey" />
-    </visual>
-    <collision>
-      <geometry>
-        <mesh filename="package://my_robot_description/meshes/left_arm/Left_forarm_lower_1.stl" scale="0.15 0.15 0.15"/>
+        <mesh filename="file:///home/shreyas/ros2_ws/src/my_robot_description/meshes/left_arm/Left_forarm_lower_1.stl" scale="0.15 0.15 0.15"/>
+      </geometry>
+      <material name="grey" />
+    </visual>
+    <collision>
+      <geometry>
+        <mesh filename="file:///home/shreyas/ros2_ws/src/my_robot_description/meshes/left_arm/Left_forarm_lower_1.stl" scale="0.15 0.15 0.15"/>
       </geometry>
     </collision>
@@ -330,11 +330,11 @@
     <visual>
       <geometry>
-        <mesh filename="package://my_robot_description/meshes/left_arm/Left_forarm_internal_support.stl" scale="0.15 0.15 0.15"/>
-      </geometry>
-      <material name="grey" />
-    </visual>
-    <collision>
-      <geometry>
-        <mesh filename="package://my_robot_description/meshes/left_arm/Left_forarm_internal_support.stl" scale="0.15 0.15 0.15"/>
+        <mesh filename="file:///home/shreyas/ros2_ws/src/my_robot_description/meshes/left_arm/Left_forarm_internal_support.stl" scale="0.15 0.15 0.15"/>
+      </geometry>
+      <material name="grey" />
+    </visual>
+    <collision>
+      <geometry>
+        <mesh filename="file:///home/shreyas/ros2_ws/src/my_robot_description/meshes/left_arm/Left_forarm_internal_support.stl" scale="0.15 0.15 0.15"/>
       </geometry>
     </collision>
@@ -356,11 +356,11 @@
     <visual>
       <geometry>
-        <mesh filename="package://my_robot_description/meshes/left_arm/left_forarm_cover.stl" scale="0.15 0.15 0.15"/>
-      </geometry>
-      <material name="grey" />
-    </visual>
-    <collision>
-      <geometry>
-        <mesh filename="package://my_robot_description/meshes/left_arm/left_forarm_cover.stl" scale="0.15 0.15 0.15"/>
+        <mesh filename="file:///home/shreyas/ros2_ws/src/my_robot_description/meshes/left_arm/left_forarm_cover.stl" scale="0.15 0.15 0.15"/>
+      </geometry>
+      <material name="grey" />
+    </visual>
+    <collision>
+      <geometry>
+        <mesh filename="file:///home/shreyas/ros2_ws/src/my_robot_description/meshes/left_arm/left_forarm_cover.stl" scale="0.15 0.15 0.15"/>
       </geometry>
     </collision>
@@ -382,5 +382,5 @@
     <visual>
       <geometry>
-        <mesh filename="package://my_robot_description/meshes/left_arm/left_wrist.stl" scale="0.15 0.15 0.15"/>
+        <mesh filename="file:///home/shreyas/ros2_ws/src/my_robot_description/meshes/left_arm/left_wrist.stl" scale="0.15 0.15 0.15"/>
       </geometry>
       <material name="orange" />
@@ -388,5 +388,5 @@
     <collision>
       <geometry>
-        <mesh filename="package://my_robot_description/meshes/left_arm/left_wrist.stl" scale="0.15 0.15 0.15"/>
+        <mesh filename="file:///home/shreyas/ros2_ws/src/my_robot_description/meshes/left_arm/left_wrist.stl" scale="0.15 0.15 0.15"/>
       </geometry>
     </collision>
@@ -411,11 +411,11 @@
     <visual>
       <geometry>
-        <mesh filename="package://my_robot_description/meshes/left_arm/left_palm.stl" scale="0.15 0.15 0.15"/>
-      </geometry>
-      <material name="grey" />
-    </visual>
-    <collision>
-      <geometry>
-        <mesh filename="package://my_robot_description/meshes/left_arm/left_palm.stl" scale="0.15 0.15 0.15"/>
+        <mesh filename="file:///home/shreyas/ros2_ws/src/my_robot_description/meshes/left_arm/left_palm.stl" scale="0.15 0.15 0.15"/>
+      </geometry>
+      <material name="grey" />
+    </visual>
+    <collision>
+      <geometry>
+        <mesh filename="file:///home/shreyas/ros2_ws/src/my_robot_description/meshes/left_arm/left_palm.stl" scale="0.15 0.15 0.15"/>
       </geometry>
     </collision>
@@ -437,11 +437,11 @@
     <visual>
       <geometry>
-        <mesh filename="package://my_robot_description/meshes/left_arm/left_thomb_to_palm.stl" scale="0.15 0.15 0.15"/>
-      </geometry>
-      <material name="grey" />
-    </visual>
-    <collision>
-      <geometry>
-        <mesh filename="package://my_robot_description/meshes/left_arm/left_thomb_to_palm.stl" scale="0.15 0.15 0.15"/>
+        <mesh filename="file:///home/shreyas/ros2_ws/src/my_robot_description/meshes/left_arm/left_thomb_to_palm.stl" scale="0.15 0.15 0.15"/>
+      </geometry>
+      <material name="grey" />
+    </visual>
+    <collision>
+      <geometry>
+        <mesh filename="file:///home/shreyas/ros2_ws/src/my_robot_description/meshes/left_arm/left_thomb_to_palm.stl" scale="0.15 0.15 0.15"/>
       </geometry>
     </collision>
@@ -463,11 +463,11 @@
     <visual>
       <geometry>
-        <mesh filename="package://my_robot_description/meshes/left_arm/left_thomb_midle.stl" scale="0.15 0.15 0.15"/>
-      </geometry>
-      <material name="grey" />
-    </visual>
-    <collision>
-      <geometry>
-        <mesh filename="package://my_robot_description/meshes/left_arm/left_thomb_midle.stl" scale="0.15 0.15 0.15"/>
+        <mesh filename="file:///home/shreyas/ros2_ws/src/my_robot_description/meshes/left_arm/left_thomb_midle.stl" scale="0.15 0.15 0.15"/>
+      </geometry>
+      <material name="grey" />
+    </visual>
+    <collision>
+      <geometry>
+        <mesh filename="file:///home/shreyas/ros2_ws/src/my_robot_description/meshes/left_arm/left_thomb_midle.stl" scale="0.15 0.15 0.15"/>
       </geometry>
     </collision>
@@ -489,5 +489,5 @@
     <visual>
       <geometry>
-        <mesh filename="package://my_robot_description/meshes/left_arm/left_thomb_upper.stl" scale="0.15 0.15 0.15"/>
+        <mesh filename="file:///home/shreyas/ros2_ws/src/my_robot_description/meshes/left_arm/left_thomb_upper.stl" scale="0.15 0.15 0.15"/>
       </geometry>
       <material name="blue" />
@@ -495,5 +495,5 @@
     <collision>
       <geometry>
-        <mesh filename="package://my_robot_description/meshes/left_arm/left_thomb_upper.stl" scale="0.15 0.15 0.15"/>
+        <mesh filename="file:///home/shreyas/ros2_ws/src/my_robot_description/meshes/left_arm/left_thomb_upper.stl" scale="0.15 0.15 0.15"/>
       </geometry>
     </collision>
@@ -515,11 +515,11 @@
     <visual>
       <geometry>
-        <mesh filename="package://my_robot_description/meshes/left_arm/left_finger1_lower.stl" scale="0.15 0.15 0.15"/>
-      </geometry>
-      <material name="grey" />
-    </visual>
-    <collision>
-      <geometry>
-        <mesh filename="package://my_robot_description/meshes/left_arm/left_finger1_lower.stl" scale="0.15 0.15 0.15"/>
+        <mesh filename="file:///home/shreyas/ros2_ws/src/my_robot_description/meshes/left_arm/left_finger1_lower.stl" scale="0.15 0.15 0.15"/>
+      </geometry>
+      <material name="grey" />
+    </visual>
+    <collision>
+      <geometry>
+        <mesh filename="file:///home/shreyas/ros2_ws/src/my_robot_description/meshes/left_arm/left_finger1_lower.stl" scale="0.15 0.15 0.15"/>
       </geometry>
     </collision>
@@ -542,11 +542,11 @@
     <visual>
       <geometry>
-        <mesh filename="package://my_robot_description/meshes/left_arm/left_finger1_middle.stl" scale="0.15 0.15 0.15"/>
-      </geometry>
-      <material name="grey" />
-    </visual>
-    <collision>
-      <geometry>
-        <mesh filename="package://my_robot_description/meshes/left_arm/left_finger1_middle.stl" scale="0.15 0.15 0.15"/>
+        <mesh filename="file:///home/shreyas/ros2_ws/src/my_robot_description/meshes/left_arm/left_finger1_middle.stl" scale="0.15 0.15 0.15"/>
+      </geometry>
+      <material name="grey" />
+    </visual>
+    <collision>
+      <geometry>
+        <mesh filename="file:///home/shreyas/ros2_ws/src/my_robot_description/meshes/left_arm/left_finger1_middle.stl" scale="0.15 0.15 0.15"/>
       </geometry>
     </collision>
@@ -569,5 +569,5 @@
     <visual>
       <geometry>
-        <mesh filename="package://my_robot_description/meshes/left_arm/left_finger1_upper.stl" scale="0.15 0.15 0.15"/>
+        <mesh filename="file:///home/shreyas/ros2_ws/src/my_robot_description/meshes/left_arm/left_finger1_upper.stl" scale="0.15 0.15 0.15"/>
       </geometry>
       <material name="blue" />
@@ -575,5 +575,5 @@
     <collision>
       <geometry>
-        <mesh filename="package://my_robot_description/meshes/left_arm/left_finger1_upper.stl" scale="0.15 0.15 0.15"/>
+        <mesh filename="file:///home/shreyas/ros2_ws/src/my_robot_description/meshes/left_arm/left_finger1_upper.stl" scale="0.15 0.15 0.15"/>
       </geometry>
     </collision>
@@ -595,11 +595,11 @@
     <visual>
       <geometry>
-        <mesh filename="package://my_robot_description/meshes/left_arm/left_finger2_lower.stl" scale="0.15 0.15 0.15"/>
-      </geometry>
-      <material name="grey" />
-    </visual>
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
Commit message: Your update message

File: src/my_robot_description/urdf/hruh.xacro (robot description, xacro)
@@ -27,5 +27,5 @@
   </joint>
   <gazebo reference="chest_hruh">
-      <material>Gazebo/Orange</material>
+      <material>Gazebo/Wood</material>
   </gazebo>
   <!-- Neck -->
