Commit message: Track large db file with Git LFS

File: src/my_robot_description/urdf/hruh.xacro (robot description, xacro)
@@ -96,1565 +96,3 @@
     </inertial>
   </link>
-  <gazebo reference="head_base">
-      <selfCollide>true</selfCollide>
-  </gazebo>
-  <!-- Left Shoulder Joint -->
-  <joint name="chest_to_left_shoulder" type="revolute">
-    <parent link="chest_hruh"/>
-    <child link="left_shoulder"/>
-    <origin xyz="0 -0.104 0.315" rpy="0 0 0"/>
-    <axis xyz="0 1 0"/>
-    <dynamics damping="1" friction="2"/>
-    <limit lower="-1.57" upper="3.14" effort="500" velocity="1.0"/>
-  </joint>
-  <link name="left_shoulder">
-    <visual>
-      <geometry>
-        <mesh filename="file:///home/shreyas/ros2_ws/src/my_robot_description/meshes/left_arm/left_S_to_C.stl" scale="0.15 0.15 0.15"/>
-      </geometry>
-      <material name="grey" />
-    </visual>
-    <collision>
-      <geometry>
-        <mesh filename="file:///home/shreyas/ros2_ws/src/my_robot_description/meshes/left_arm/left_S_to_C.stl" scale="0.15 0.15 0.15"/>
-      </geometry>
-    </collision>
-    <inertial>
-      <mass value="1.2"/>
-      <inertia ixx="0.004" ixy="0.0" ixz="0.0" iyy="0.004" iyz="0.0" izz="0.003"/>
-      <origin xyz="0 0 0" rpy="0 0 0"/>
-    </inertial>
-  </link>
-  <gazebo reference="left_shoulder">
-      <selfCollide>true</selfCollide>
-  </gazebo>
-  <!-- Left S to bisecp Arm Joint -->
-  <joint name="left_shoulder_to_bisecp" type="revolute">
-    <parent link="left_shoulder"/>
-    <child link="left_S_to_Bisecp"/>
-    <origin xyz="0.01 -0.0795 0.02" rpy="0 0 0"/>
-    <axis xyz="1 0 0"/>
-    <dynamics damping="1" friction="2"/>
-    <limit lower="-1.57" upper="0.45" effort="500" velocity="1.0"/>
-  </joint>
-  <link name="left_S_to_Bisecp">
-    <visual>
-      <geometry>
-        <mesh filename="file:///home/shreyas/ros2_ws/src/my_robot_description/meshes/left_arm/left_S_to_Bisecp.stl" scale="0.15 0.15 0.15"/>
-      </geometry>
-      <material name="grey" />
-    </visual>
-    <collision>
-      <geometry>
-        <mesh filename="file:///home/shreyas/ros2_ws/src/my_robot_description/meshes/left_arm/left_S_to_Bisecp.stl" scale="0.15 0.15 0.15"/>
-      </geometry>
-    </collision>
-    <inertial>
-      <mass value="1.5"/>
-      <inertia ixx="0.005" ixy="0.0" ixz="0.0" iyy="0.0045" iyz="0.0" izz="0.0035"/>
-      <origin xyz="0 0 0" rpy="0 0 0"/>
-    </inertial>
-  </link>
-  <gazebo reference="left_S_to_Bisecp">
-      <selfCollide>true</selfCollide>
-  </gazebo>
-  <!-- Left Bisecp uper Joint -->
-  <joint name="left_S_to_bisecp_upper" type="fixed">
-    <parent link="left_S_to_Bisecp"/>
-    <child link="left_bisecp_upper"/>
-    <origin xyz="-0.007 0.0025 -0.095" rpy="0 0 0"/>
-    <axis xyz="0 0 0"/>
-    <limit lower="-1.57" upper="1.57" effort="500" velocity="1.0"/>
-  </joint>
-  <link name="left_bisecp_upper">
-    <visual>
-      <geometry>
-        <mesh filename="file:///home/shreyas/ros2_ws/src/my_robot_description/meshes/left_arm/Left_bisecp_uper.stl" scale="0.15 0.15 0.15"/>
-      </geometry>
-      <material name="grey" />
-    </visual>
-    <collision>
-      <geometry>
-        <mesh filename="file:///home/shreyas/ros2_ws/src/my_robot_description/meshes/left_arm/Left_bisecp_uper.stl" scale="0.15 0.15 0.15"/>
-      </geometry>
-    </collision>
-    <inertial>
-      <mass value="0.9"/>
-      <inertia ixx="0.003" ixy="0.0" ixz="0.0" iyy="0.0025" iyz="0.0" izz="0.002"/>
-      <origin xyz="0 0 0" rpy="0 0 0"/>
-    </inertial>
-  </link>
-  <gazebo reference="left_bisecp_upper">
-      <selfCollide>true</selfCollide>
-  </gazebo>
-  <!-- Left Bisecp lower Joint -->
-  <joint name="left_bisecp_uper_to_lower" type="fixed">
-    <parent link="left_bisecp_upper"/>
-    <child link="left_bisecp_lower"/>
-    <origin xyz="0 0 -0.042" rpy="0 0 0"/>
-    <axis xyz="0 0 0"/>
-    <limit lower="-1.57" upper="1.57" effort="500" velocity="1.0"/>
-  </joint>
-  <link name="left_bisecp_lower">
-    <visual>
-      <geometry>
-        <mesh filename="file:///home/shreyas/ros2_ws/src/my_robot_description/meshes/left_arm/left_Bisecp_lower.stl" scale="0.15 0.15 0.15"/>
-      </geometry>
-      <material name="grey" />
-    </visual>
-    <collision>
-      <geometry>
-        <mesh filename="file:///home/shreyas/ros2_ws/src/my_robot_description/meshes/left_arm/left_Bisecp_lower.stl" scale="0.15 0.15 0.15"/>
-      </geometry>
-    </collision>
-    <inertial>
-      <mass value="0.8"/>
-      <inertia ixx="0.0025" ixy="0.0" ixz="0.0" iyy="0.0025" iyz="0.0" izz="0.0018"/>
-      <origin xyz="0 0 0" rpy="0 0 0"/>
-    </inertial>
-  </link>
-  <gazebo reference="left_bisecp_lower">
-      <selfCollide>true</selfCollide>
-  </gazebo>
-  <!-- Left elbow inword Joint -->
-  <joint name="left_bisecp_to_elbow_inword" type="revolute">
-    <parent link="left_bisecp_lower"/>
-    <child link="left_elbow_inword"/>
-    <origin xyz="0. 0 -0.12" rpy="0 0 0"/>
-    <axis xyz="0 0 1"/>
-    <dynamics damping="1" friction="2"/>
-    <limit lower="-1.57" upper="1.57" effort="500" velocity="1.0"/>
-  </joint>
-  <link name="left_elbow_inword">
-    <visual>
-      <geometry>
-        <mesh filename="file:///home/shreyas/ros2_ws/src/my_robot_description/meshes/left_arm/left_elbow_inword.stl" scale="0.15 0.15 0.15"/>
-      </geometry>
-      <material name="grey" />
-    </visual>
-    <collision>
-      <geometry>
-        <mesh filename="file:///home/shreyas/ros2_ws/src/my_robot_description/meshes/left_arm/left_elbow_inword.stl" scale="0.15 0.15 0.15"/>
-      </geometry>
-    </collision>
-    <inertial>
-      <mass value="0.6"/>
-      <inertia ixx="0.002" ixy="0.0" ixz="0.0" iyy="0.0018" iyz="0.0" izz="0.0015"/>
-      <origin xyz="0 0 0" rpy="0 0 0"/>
-    </inertial>
-  </link>
-  <gazebo reference="left_elbow_inword">
-      <selfCollide>true</selfCollide>
-  </gazebo>
-  <!-- Left elbow midle Joint -->
-  <joint name="left_elbow_inword_to_midle" type="revolute">
-    <parent link="left_elbow_inword"/>
-    <child link="left_elbow_midle"/>
-    <origin xyz="0 -0.012 0" rpy="0 0 0"/>
-    <axis xyz="0 1 0"/>
-    <dynamics damping="1" friction="2"/>
-    <limit lower="0" upper="1.9" effort="500" velocity="1.0"/>
-  </joint>
-  <link name="left_elbow_midle">
-    <visual>
-      <geometry>
-        <mesh filename="file:///home/shreyas/ros2_ws/src/my_robot_description/meshes/left_arm/left_elbow_midle.stl" scale="0.15 0.15 0.15"/>
-      </geometry>
-      <material name="grey" />
-    </visual>
-    <collision>
-      <geometry>
-        <mesh filename="file:///home/shreyas/ros2_ws/src/my_robot_description/meshes/left_arm/left_elbow_midle.stl" scale="0.15 0.15 0.15"/>
-      </geometry>
-    </collision>
-    <inertial>
-      <mass value="0.6"/>
-      <inertia ixx="0.002" ixy="0.0" ixz="0.0" iyy="0.0018" iyz="0.0" izz="0.0015"/>
-      <origin xyz="0 0 0" rpy="0 0 0"/>
-    </inertial>
-  </link>
-  <gazebo reference="left_elbow_midle">
-      <selfCollide>true</selfCollide>
-  </gazebo>
-  <!-- Left elbow outword Joint -->
-  <joint name="left_elbow_midle_to_outword" type="fixed">
-    <parent link="left_elbow_midle"/>
-    <child link="Left_elbow_outword"/>
-    <origin xyz="0 -0.0175 0" rpy="0 0 0"/>
-    <axis xyz="0 0 0"/>
-    <limit lower="-1.57" upper="1.57" effort="500" velocity="1.0"/>
-  </joint>
-  <link name="Left_elbow_outword">
-    <visual>
-      <geometry>
-        <mesh filename="file:///home/shreyas/ros2_ws/src/my_robot_description/meshes/left_arm/Left_elbow_outword.stl" scale="0.15 0.15 0.15"/>
-      </geometry>
-      <material name="grey" />
-    </visual>
-    <collision>
-      <geometry>
-        <mesh filename="file:///home/shreyas/ros2_ws/src/my_robot_description/meshes/left_arm/Left_elbow_outword.stl" scale="0.15 0.15 0.15"/>
-      </geometry>
-    </collision>
-    <inertial>
-      <mass value="0.5"/>
-      <inertia ixx="0.0015" ixy="0.0" ixz="0.0" iyy="0.0015" iyz="0.0" izz="0.0012"/>
-      <origin xyz="0 0 0" rpy="0 0 0"/>
-    </inertial>
-  </link>
-  <gazebo reference="left_elbow_outword">
-      <selfCollide>true</selfCollide>
-  </gazebo>
-  <!-- Left elbow to forarm upper Joint -->
-  <joint name="left_elbow_midle_forarm_upper" type="fixed">
-    <parent link="left_elbow_midle"/>
-    <child link="left_elbow_to_forarm_upper"/>
-    <origin xyz="0 0.0065 -0.0645" rpy="0 0 0"/>
-    <axis xyz="0 0 0"/>
-    <limit lower="-1.57" upper="1.57" effort="500" velocity="1.0"/>
-  </joint>
-  <link name="left_elbow_to_forarm_upper">
-    <visual>
-      <geometry>
-        <mesh filename="file:///home/shreyas/ros2_ws/src/my_robot_description/meshes/left_arm/left_elbow_to_forarm_upper.stl" scale="0.15 0.15 0.15"/>
-      </geometry>
-      <material name="grey" />
-    </visual>
-    <collision>
-      <geometry>
-        <mesh filename="file:///home/shreyas/ros2_ws/src/my_robot_description/meshes/left_arm/left_elbow_to_forarm_upper.stl" scale="0.15 0.15 0.15"/>
-      </geometry>
-    </collision>
-    <inertial>
-      <mass value="0.8"/>
-      <inertia ixx="0.0025" ixy="0.0" ixz="0.0" iyy="0.002" iyz="0.0" izz="0.002"/>
-      <origin xyz="0 0 0" rpy="0 0 0"/>
-    </inertial>
-  </link>
-  <gazebo reference="left_elbow_to_forarm_upper">
-      <selfCollide>true</selfCollide>
-  </gazebo>
-  <!-- Left forarm upper to lower Joint -->
-  <joint name="left_forarm_upper_to_lower_1" type="fixed">
-    <parent link="left_elbow_to_forarm_upper"/>
-    <child link="Left_forarm_lower_1"/>
-    <origin xyz="0 0 -0.04" rpy="0 0 0"/>
-    <axis xyz="0 0 0"/>
-    <limit lower="-1.57" upper="1.57" effort="500" velocity="1.0"/>
-  </joint>
-  <link name="Left_forarm_lower_1">
-    <visual>
-      <geometry>
-        <mesh filename="file:///home/shreyas/ros2_ws/src/my_robot_description/meshes/left_arm/Left_forarm_lower_1.stl" scale="0.15 0.15 0.15"/>
-      </geometry>
-      <material name="grey" />
-    </visual>
-    <collision>
-      <geometry>
-        <mesh filename="file:///home/shreyas/ros2_ws/src/my_robot_description/meshes/left_arm/Left_forarm_lower_1.stl" scale="0.15 0.15 0.15"/>
-      </geometry>
-    </collision>
-    <inertial>
-      <mass value="0.7"/>
-      <inertia ixx="0.002" ixy="0.0" ixz="0.0" iyy="0.002" iyz="0.0" izz="0.0015"/>
-      <origin xyz="0 0 0" rpy="0 0 0"/>
-    </inertial>
-  </link>
-  <gazebo reference="left_forarm_lower_1">
-      <selfCollide>true</selfCollide>
-  </gazebo>
-  <!-- Left forarm internal support -->
-  <joint name="left_forarm_lower_1_to_internal_support" type="fixed">
-    <parent link="Left_forarm_lower_1"/>
-    <child link="Left_forarm_internal_support"/>
-    <origin xyz="0 -0.001 -0.05185" rpy="0 0 0"/>
-    <axis xyz="0 0 0"/>
-    <limit lower="-1.57" upper="1.57" effort="500" velocity="1.0"/>
-  </joint>
-  <link name="Left_forarm_internal_support">
-    <visual>
-      <geometry>
-        <mesh filename="file:///home/shreyas/ros2_ws/src/my_robot_description/meshes/left_arm/Left_forarm_internal_support.stl" scale="0.15 0.15 0.15"/>
-      </geometry>
-      <material name="grey" />
-    </visual>
-    <collision>
-      <geometry>
-        <mesh filename="file:///home/shreyas/ros2_ws/src/my_robot_description/meshes/left_arm/Left_forarm_internal_support.stl" scale="0.15 0.15 0.15"/>
-      </geometry>
-    </collision>
-    <inertial>
-      <mass value="0.3"/>
-      <inertia ixx="0.001" ixy="0.0" ixz="0.0" iyy="0.001" iyz="0.0" izz="0.001"/>
-      <origin xyz="0 0 0" rpy="0 0 0"/>
-    </inertial>
-  </link>
-  <gazebo reference="left_forarm_internal_support">
-      <selfCollide>true</selfCollide>
-  </gazebo>
-  <!-- Left forarm cover joint -->
-  <joint name="left_internal_support_to_cover" type="fixed">
-    <parent link="Left_forarm_internal_support"/>
-    <child link="left_forarm_cover"/>
-    <origin xyz="0 0.001 -0.001" rpy="0 0 0"/>
-    <axis xyz="0 0 0"/>
-    <limit lower="-1.57" upper="1.57" effort="500" velocity="1.0"/>
-  </joint>
-  <link name="left_forarm_cover">
-    <visual>
-      <geometry>
-        <mesh filename="file:///home/shreyas/ros2_ws/src/my_robot_description/meshes/left_arm/left_forarm_cover.stl" scale="0.15 0.15 0.15"/>
-      </geometry>
-      <material name="grey" />
-    </visual>
-    <collision>
-      <geometry>
-        <mesh filename="file:///home/shreyas/ros2_ws/src/my_robot_description/meshes/left_arm/left_forarm_cover.stl" scale="0.15 0.15 0.15"/>
-      </geometry>
-    </collision>
-    <inertial>
-      <mass value="0.2"/>
-      <inertia ixx="0.0005" ixy="0.0" ixz="0.0" iyy="0.0005" iyz="0.0" izz="0.0005"/>
-      <origin xyz="0 0 0" rpy="0 0 0"/>
-    </inertial>
-  </link>
-  <gazebo reference="left_forarm_cover">
-      <selfCollide>true</selfCollide>
-  </gazebo>
-  <!-- Left bisecp to wrist Joint -->
-  <joint name="left_forarm_to_wrist" type="revolute">
-    <parent link="Left_forarm_internal_support"/>
-    <child link="left_wrist"/>
-    <origin xyz="0 0.0015 -0.061" rpy="0 0 0"/>
-    <axis xyz="0 0 1"/>
-    <dynamics damping="1" friction="2"/>
-    <limit lower="-1.57" upper="1.57" effort="500" velocity="1.0"/>
-  </joint>
-  <link name="left_wrist">
-    <visual>
-      <geometry>
-        <mesh filename="file:///home/shreyas/ros2_ws/src/my_robot_description/meshes/left_arm/left_wrist.stl" scale="0.15 0.15 0.15"/>
-      </geometry>
-      <material name="orange" />
-    </visual>
-    <collision>
-      <geometry>
-        <mesh filename="file:///home/shreyas/ros2_ws/src/my_robot_description/meshes/left_arm/left_wrist.stl" scale="0.15 0.15 0.15"/>
-      </geometry>
-    </collision>
-    <inertial>
-      <mass value="0.4"/>
-      <inertia ixx="0.001" ixy="0.0" ixz="0.0" iyy="0.001" iyz="0.0" izz="0.0008"/>
-      <origin xyz="0 0 0" rpy="0 0 0"/>
-    </inertial>
-  </link>
-  <gazebo reference="left_wrist">
-      <material>Gazebo/Orange</material>
-  </gazebo>
-  <gazebo reference="left_wrist">
-      <material>Gazebo/Orange</material>
-  </gazebo>
-  <!-- Left palm joint -->
-  <joint name="left_wrist_to_palm" type="fixed">
-    <parent link="left_wrist"/>
-    <child link="left_palm"/>
-    <origin xyz="0 0 -0.04" rpy="0 0 0"/>
-    <axis xyz="0 0 0"/>
-    <limit lower="-1.57" upper="1.57" effort="500" velocity="1.0"/>
-  </joint>
-  <link name="left_palm">
-    <visual>
-      <geometry>
-        <mesh filename="file:///home/shreyas/ros2_ws/src/my_robot_description/meshes/left_arm/left_palm.stl" scale="0.15 0.15 0.15"/>
-      </geometry>
-      <material name="grey" />
-    </visual>
-    <collision>
-      <geometry>
-        <mesh filename="file:///home/shreyas/ros2_ws/src/my_robot_description/meshes/left_arm/left_palm.stl" scale="0.15 0.15 0.15"/>
-      </geometry>
-    </collision>
-    <inertial>
-      <mass value="0.5"/>
-      <inertia ixx="0.0015" ixy="0.0" ixz="0.0" iyy="0.0015" iyz="0.0" izz="0.001"/>
-      <origin xyz="0 0 0" rpy="0 0 0"/>
-    </inertial>
-  </link>
-  <gazebo reference="left_palm">
-      <selfCollide>true</selfCollide>
-  </gazebo>
-  <!-- Left palm to thomb joint -->
-  <joint name="left_palm_to_thomb" type="revolute">
-    <parent link="left_palm"/>
-    <child link="left_thomb_to_palm"/>
-    <origin xyz="-0.021 0 0.018" rpy="0 0 0"/>
-    <axis xyz="0 0 1"/>
-    <dynamics damping="1" friction="2"/>
-    <limit lower="-1.8" upper="0" effort="500" velocity="1.0"/>
-  </joint>
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
File: src/my_robot_description/urdf/hruh_gazebo.xacro (robot description, xacro)
@@ -41,53 +41,4 @@
       <i_min>-6</i_min><i_max>6</i_max>
     </plugin>
-    <!-- Left palm to thomb joint -->
-    <plugin filename="gz-sim-joint-position-controller-system"
-        name="gz::sim::systems::JointPositionController">
-      <joint_name>left_palm_to_thomb</joint_name>
-      <p_gain>300</p_gain><i_gain>2</i_gain><d_gain>3</d_gain>
-      <i_min>-6</i_min><i_max>6</i_max>
-    </plugin>
-    <!-- left_thomb_to_thomb_middle -->
-    <plugin filename="gz-sim-joint-position-controller-system"
-        name="gz::sim::systems::JointPositionController">
-      <joint_name>left_thomb_to_thomb_middle</joint_name>
-      <p_gain>300</p_gain><i_gain>2</i_gain><d_gain>3</d_gain>
-      <i_min>-6</i_min><i_max>6</i_max>
-    </plugin>
-    <!-- left_thomb_middle_to_thomb_upper -->
-    <plugin filename="gz-sim-joint-position-controller-system"
-        name="gz::sim::systems::JointPositionController">
-      <joint_name>left_thomb_middle_to_thomb_upper</joint_name>
-      <p_gain>300</p_gain><i_gain>2</i_gain><d_gain>3</d_gain>
-      <i_min>-6</i_min><i_max>6</i_max>
-    </plugin>
-    <!-- Left palm  to finger1 lower -->
-    <plugin filename="gz-sim-joint-position-controller-system"
-        name="gz::sim::systems::JointPositionController">
-      <joint_name>left_palm_to_finger1_lower</joint_name>
-      <p_gain>300</p_gain><i_gain>2</i_gain><d_gain>3</d_gain>
-      <i_min>-6</i_min><i_max>6</i_max>
-    </plugin>
-    <!-- Left palm  to finger2 lower -->
-    <plugin filename="gz-sim-joint-position-controller-system"
-        name="gz::sim::systems::JointPositionController">
-      <joint_name>left_palm_to_finger2_lower</joint_name>
-      <p_gain>300</p_gain><i_gain>2</i_gain><d_gain>3</d_gain>
-      <i_min>-6</i_min><i_max>6</i_max>
-    </plugin>
-    <!-- Left palm  to finger3 lower -->
-    <plugin filename="gz-sim-joint-position-controller-system"
-        name="gz::sim::systems::JointPositionController">
-      <joint_name>left_palm_to_finger3_lower</joint_name>
-      <p_gain>300</p_gain><i_gain>2</i_gain><d_gain>3</d_gain>
-      <i_min>-6</i_min><i_max>6</i_max>
-    </plugin>
-    <!-- Left palm  to finger4 lower -->
-    <plugin filename="gz-sim-joint-position-controller-system"
-            name="gz::sim::systems::JointPositionController">
-      <joint_name>left_palm_to_finger4_lower</joint_name>
-      <p_gain>300</p_gain><i_gain>2</i_gain><d_gain>3</d_gain>
-      <i_min>-6</i_min><i_max>6</i_max>
-    </plugin>
     <!-- repeat per joint ... -->
   </gazebo>
@@ -128,53 +79,4 @@
       <i_min>-6</i_min><i_max>6</i_max>
     </plugin>
-    <!-- right palm to thomb joint -->
-    <plugin filename="gz-sim-joint-position-controller-system"
-        name="gz::sim::systems::JointPositionController">
-      <joint_name>right_palm_to_thomb</joint_name>
-      <p_gain>300</p_gain><i_gain>2</i_gain><d_gain>3</d_gain>
-      <i_min>-6</i_min><i_max>6</i_max>
-    </plugin>
-    <!-- tright_thomb_to_thomb_middle -->
-    <plugin filename="gz-sim-joint-position-controller-system"
-        name="gz::sim::systems::JointPositionController">
-      <joint_name>right_thomb_to_thomb_middle</joint_name>
-      <p_gain>300</p_gain><i_gain>2</i_gain><d_gain>3</d_gain>
-      <i_min>-6</i_min><i_max>6</i_max>
-    </plugin>
-    <!-- right_thomb_middle_to_thomb_upper -->
-    <plugin filename="gz-sim-joint-position-controller-system"
-        name="gz::sim::systems::JointPositionController">
-      <joint_name>right_thomb_middle_to_thomb_upper</joint_name>
-      <p_gain>300</p_gain><i_gain>2</i_gain><d_gain>3</d_gain>
-      <i_min>-6</i_min><i_max>6</i_max>
-    </plugin>
-    <!-- right palm  to finger1 lower -->
-    <plugin filename="gz-sim-joint-position-controller-system"
-        name="gz::sim::systems::JointPositionController">
-      <joint_name>right_palm_to_finger1_lower</joint_name>
-      <p_gain>300</p_gain><i_gain>2</i_gain><d_gain>3</d_gain>
-      <i_min>-6</i_min><i_max>6</i_max>
-    </plugin>
-    <!-- right palm  to finger2 lower -->
-    <plugin filename="gz-sim-joint-position-controller-system"
-        name="gz::sim::systems::JointPositionController">
-      <joint_name>right_palm_to_finger2_lower</joint_name>
-      <p_gain>300</p_gain><i_gain>2</i_gain><d_gain>3</d_gain>
-      <i_min>-6</i_min><i_max>6</i_max>
-    </plugin>
-    <!-- right palm  to finger3 lower -->
-    <plugin filename="gz-sim-joint-position-controller-system"
-        name="gz::sim::systems::JointPositionController">
-      <joint_name>right_palm_to_finger3_lower</joint_name>
-      <p_gain>300</p_gain><i_gain>2</i_gain><d_gain>3</d_gain>
-      <i_min>-6</i_min><i_max>6</i_max>
-    </plugin>
-    <!-- right palm  to finger4 lower -->
-    <plugin filename="gz-sim-joint-position-controller-system"
-            name="gz::sim::systems::JointPositionController">
-      <joint_name>right_palm_to_finger4_lower</joint_name>
-      <p_gain>300</p_gain><i_gain>2</i_gain><d_gain>3</d_gain>
-      <i_min>-6</i_min><i_max>6</i_max>
-    </plugin>
     <!-- repeat per joint ... -->
   </gazebo>

File: src/my_robot_description/urdf/my_robot.urdf.xacro (robot description, xacro)
@@ -10,4 +10,8 @@
     <xacro:include filename="camera.xacro" />
     <xacro:include filename="lidar.xacro" />
+    <xacro:include filename="right_arm.xacro" />
+    <xacro:include filename="right_arm_gripper.xacro" />
+    <xacro:include filename="left_arm.xacro" />
+    <xacro:include filename="left_arm_gripper.xacro" />
     <joint name="mobile_base_arm_joint" type="fixed">
         <parent link="base_link" />
@@ -15,6 +19,3 @@
         <origin xyz="${base_length / 10.0} 0 ${base_height}" rpy="0 0 3.14" />
     </joint>
-    <gazebo>
-        <selfCollide>true</selfCollide>
-    </gazebo>
 </robot>
