Commit message: commit

File: src/my_robot_description/urdf/lidar_gz.xacro (robot description, xacro)
@@ -3,5 +3,5 @@
   <!-- simple mast link for LiDAR -->
   <link name="lidar_link">
-    <visual>
+    <!-- <visual>
       <geometry><cylinder radius="0.035" length="0.06"/></geometry>
       <material name="grey"/>
@@ -15,5 +15,5 @@
       <origin xyz="0 0 0" rpy="0 0 0"/>
       <inertia ixx="1e-4" ixy="0" ixz="0" iyy="1e-4" iyz="0" izz="1e-4"/>
-    </inertial>
+    </inertial> -->
   </link>
   <!-- mount LiDAR somewhere reasonable above base_link -->

File: src/my_robot_description/urdf/mobile_base.xacro (robot description, xacro)
@@ -65,5 +65,4 @@
         <origin xyz="${(base_length) / 4.0} ${-(base_width + wheel_length) / 2.0} 0" rpy="0 0 0" />
         <axis xyz="0 1 0" />
-        <mimic joint="base_right_back_wheel_joint" multiplier="1" />
     </joint>
      <joint name="base_left_back_wheel_joint" type="continuous">
@@ -78,5 +77,4 @@
         <origin xyz="${base_length / 4.0} ${(base_width + wheel_length) / 2.0} 0" rpy="0 0 0" />
         <axis xyz="0 1 0" />
-        <mimic joint="base_left_back_wheel_joint" multiplier="1" />
     </joint>
     <joint name="base_footprint_joint" type="fixed">

File: src/my_robot_description/urdf/mobile_base_gazebo.xacro (robot description, xacro)
@@ -46,6 +46,10 @@
             <wheel_separation>0.45</wheel_separation>
             <wheel_radius>0.1</wheel_radius>
+            <topic>/model/my_robot/cmd_vel</topic>
+            <odom_topic>/model/my_robot/odometry</odom_topic>
+            <tf_topic>/model/my_robot/tf</tf_topic>
             <frame_id>odom</frame_id>
             <child_frame_id>base_footprint</child_frame_id>
+            <odom_publish_frequency>30</odom_publish_frequency>
         </plugin>
     </gazebo>
