Commit message: commit

File: src/my_robot_description/urdf/hruh.ros2_control.xacro (robot description, xacro)
@@ -6,10 +6,11 @@
                   state, for MoveIt / RViz without a simulator
   hardware:=none  no ros2_control (e.g. joint_state_publisher_gui display)
-  Controllers: config/ros2_controllers.yaml
+  Controllers: hruh_control/config/ros2_controllers.yaml
     legs_controller        14 leg joints, streamed by hruh_walker
     waist_controller       3-DOF waist        (JointTrajectoryController)
     head_controller        neck yaw + nod     (JointTrajectoryController)
     left/right_arm_controller   5 joints each (MoveIt, servo, joystick)
-    left/right_hand_controller 15 joints each (open / close grasp)
+    left/right_hand_controller 7 joints each: thumb x3 + finger base x4
+                          (middle / upper finger joints are URDF mimic joints)
 -->
 <robot xmlns:xacro="http://www.ros.org/wiki/xacro">
@@ -21,7 +22,9 @@
          'chest_to_right_shoulder', 'right_shoulder_to_bisecp', 'right_bisecp_to_elbow_inword', 'right_elbow_inword_to_midle', 'right_forarm_to_wrist']
       + [s + '_' + n for s in ['left', 'right'] for n in ['palm_to_thomb', 'thomb_to_thomb_middle', 'thomb_middle_to_thomb_upper']
-                                                         + ['palm_to_finger%d_lower' % i for i in [1, 2, 3, 4]]
-                                                         + ['finger%d_lower_to_finger%d_middle' % (i, i) for i in [1, 2, 3, 4]]
-                                                         + ['finger%d_middle_to_finger%d_upper' % (i, i) for i in [1, 2, 3, 4]]]}"/>
+                                                         + ['palm_to_finger%d_lower' % i for i in [1, 2, 3, 4]]]}"/>
+  <!-- middle / upper finger joints mimic the lower one (URDF <mimic>): state only -->
+  <xacro:property name="hruh_mimic_joints" value="${[s + '_' + n for s in ['left', 'right']
+                                                     for n in ['finger%d_lower_to_finger%d_middle' % (i, i) for i in [1, 2, 3, 4]]
+                                                            + ['finger%d_middle_to_finger%d_upper' % (i, i) for i in [1, 2, 3, 4]]]}"/>
   <xacro:macro name="hruh_ctrl_joint" params="name">
     <joint name="${name}">
@@ -32,4 +35,16 @@
       <state_interface name="velocity"/>
     </joint>
+  </xacro:macro>
+  <xacro:macro name="hruh_mimic_joint" params="name">
+    <joint name="${name}">
+      <state_interface name="position"/>
+      <state_interface name="velocity"/>
+    </joint>
+  </xacro:macro>
+  <xacro:macro name="hruh_mimic_joints" params="names">
+    <xacro:if value="${len(names) > 0}">
+      <xacro:hruh_mimic_joint name="${names[0]}"/>
+      <xacro:hruh_mimic_joints names="${names[1:]}"/>
+    </xacro:if>
   </xacro:macro>
   <xacro:macro name="hruh_ctrl_joints" params="names">
@@ -51,10 +66,14 @@
       </hardware>
       <xacro:hruh_ctrl_joints names="${hruh_leg_joints + hruh_upper_joints}"/>
+      <xacro:hruh_mimic_joints names="${hruh_mimic_joints}"/>
     </ros2_control>
   </xacro:unless>
   <xacro:if value="${hardware == 'gz'}">
     <gazebo>
+      <!-- controller config lives in hruh_control (see the note at the top of that file) -->
       <plugin filename="gz_ros2_control-system" name="gz_ros2_control::GazeboSimROS2ControlPlugin">
-        <parameters>$(find my_robot_description)/config/ros2_controllers.yaml</parameters>
+        <parameters>$(find hruh_control)/config/ros2_controllers.yaml</parameters>
+        <robot_param>robot_description</robot_param>
+        <robot_param_node>robot_state_publisher</robot_param_node>
       </plugin>
     </gazebo>

Commit message: commit

File: src/my_robot_description/urdf/hruh.ros2_control.xacro (robot description, xacro)
@@ -9,6 +9,6 @@
   hardware:=none  no ros2_control (e.g. joint_state_publisher_gui display)
   Controllers: hruh_control/config/ros2_controllers.yaml
-    legs_controller        14 leg joints, streamed by hruh_walker
-    waist_controller       3-DOF waist        (JointTrajectoryController)
+    legs_controller        14 leg joints, streamed by hruh_walker / the walking policy
+    (the torso is rigid: no waist joints)
     head_controller        neck yaw + nod     (JointTrajectoryController)
     left/right_arm_controller   5 joints each (MoveIt, servo, joystick)
@@ -20,5 +20,5 @@
   <xacro:property name="hardware" value="$(arg hardware)"/>
   <xacro:property name="hruh_leg_joints" value="${[s + '_' + j + '_joint' for s in ['left', 'right'] for j in ['hip_yaw', 'hip_roll', 'hip_pitch', 'knee', 'ankle_pitch', 'ankle_roll', 'toe']]}"/>
-  <xacro:property name="hruh_upper_joints" value="${['waist_yaw_joint', 'waist_roll_joint', 'waist_pitch_joint', 'chest_to_neck', 'neck_to_head']
+  <xacro:property name="hruh_upper_joints" value="${['chest_to_neck', 'neck_to_head']
       + ['chest_to_left_shoulder', 'left_shoulder_to_bisecp', 'left_bisecp_to_elbow_inword', 'left_elbow_inword_to_midle', 'left_forarm_to_wrist',
          'chest_to_right_shoulder', 'right_shoulder_to_bisecp', 'right_bisecp_to_elbow_inword', 'right_elbow_inword_to_midle', 'right_forarm_to_wrist']

File: src/my_robot_description/urdf/legs.xacro (robot description, xacro)
@@ -3,5 +3,8 @@
   HRUH lower body: pelvis + two 7-DOF legs.
   Kinematics follow the human leg:
-    hip   : yaw (z) -> roll (x) -> pitch (y), all three axes meet at the hip centre (ball joint)
+    hip   : yaw (z) -> roll (x) -> pitch (y), all three axes meet at the hip centre (ball joint).
+            The actuators sit along their own axes where they physically fit (blender HIP):
+            yaw motor inside the pelvis above the hip, roll motor behind the hip centre,
+            pitch motor outside the thigh. Link masses / centres of mass follow the motors.
     knee  : pitch (y), flexion positive
     ankle : pitch (y) -> roll (x), axes meet at the ankle centre
@@ -12,5 +15,5 @@
 <robot xmlns:xacro="http://www.ros.org/wiki/xacro">
   <!-- Geometry (keep in sync with KIN in blender/build_parts.py) -->
-  <xacro:property name="hip_y"        value="0.085"/>
+  <xacro:property name="hip_y"        value="0.105"/>  <!-- 0.085 let the thighs collide -->
   <xacro:property name="hip_yaw_z"    value="-0.03"/>
   <xacro:property name="hip_roll_z"   value="-0.06"/>
@@ -55,8 +58,9 @@
     <xacro:mesh_visual file="pelvis.obj"/>
     <collision>
-      <origin xyz="0 0 0.01" rpy="0 0 0"/>
-      <geometry><box size="0.18 0.26 0.10"/></geometry>
+      <origin xyz="0 0 0.03" rpy="0 0 0"/>
+      <geometry><box size="0.18 0.30 0.09"/></geometry>
     </collision>
-    <xacro:solid_box_inertial m="7.0" x="0.18" y="0.28" z="0.12" oz="0.005"/>
+    <!-- shell, battery and both hip-yaw actuators -->
+    <xacro:solid_box_inertial m="9.0" x="0.18" y="0.30" z="0.10" oz="0.015"/>
   </link>
   <joint name="base_pelvis_joint" type="fixed">
@@ -74,5 +78,6 @@
   <!-- side: left|right, s: +1 (left) / -1 (right) -->
   <xacro:macro name="hruh_leg" params="side s">
-    <!-- Hip yaw: internal/external rotation (~40 / 45 deg) -->
+    <!-- Hip yaw: internal/external rotation 40 / 43 deg (one leg reaches its mechanism limit at 45;
+         both feet toed out > 21 deg make the rear roll actuators touch: self-collision) -->
     <joint name="${side}_hip_yaw_joint" type="revolute">
       <parent link="pelvis_link"/>
@@ -80,12 +85,19 @@
       <origin xyz="0 ${s*hip_y} ${hip_yaw_z}" rpy="0 0 0"/>
       <axis xyz="0 0 1"/>
-      <limit lower="${-0.70 if s > 0 else -0.79}" upper="${0.79 if s > 0 else 0.70}" effort="150" velocity="8.0"/>
+      <limit lower="${-0.70 if s > 0 else -0.75}" upper="${0.75 if s > 0 else 0.70}" effort="150" velocity="8.0"/>
       <dynamics damping="0.5" friction="0.1"/>
     </joint>
     <link name="${side}_hip_yaw_link">
       <xacro:mesh_visual file="${side}_hip_yaw.obj"/>
-      <xacro:solid_cyl_inertial m="1.4" r="0.045" h="0.06" oz="-0.03"/>
-    </link>
-    <!-- Hip roll: abduction 45 deg / adduction 25 deg -->
+      <!-- carries the hip roll actuator, 13 cm behind the hip centre -->
+      <collision>
+        <origin xyz="-0.130 0 ${hip_roll_z}" rpy="0 ${pi/2} 0"/>
+        <geometry><cylinder radius="0.050" length="0.055"/></geometry>
+      </collision>
+      <xacro:solid_cyl_inertial m="2.7" r="0.05" h="0.06" ox="-0.115" oz="-0.055"/>
+    </link>
+    <!-- Hip roll: abduction 31 deg / adduction 24 deg. Measured on the meshes (blender/design check):
+         the pitch actuator meets the pelvis at 33 deg abduction; the hip itself allows 25 deg
+         adduction (the other leg may be touched before that: self-collision) -->
     <joint name="${side}_hip_roll_joint" type="revolute">
       <parent link="${side}_hip_yaw_link"/>
@@ -93,12 +105,18 @@
       <origin xyz="0 0 ${hip_roll_z}" rpy="0 0 0"/>
       <axis xyz="1 0 0"/>
-      <limit lower="${-0.44 if s > 0 else -0.79}" upper="${0.79 if s > 0 else 0.44}" effort="200" velocity="8.0"/>
+      <limit lower="${-0.42 if s > 0 else -0.54}" upper="${0.54 if s > 0 else 0.42}" effort="200" velocity="8.0"/>
       <dynamics damping="0.5" friction="0.1"/>
     </joint>
     <link name="${side}_hip_roll_link">
       <xacro:mesh_visual file="${side}_hip_roll.obj"/>
-      <xacro:solid_box_inertial m="1.8" x="0.11" y="0.09" z="0.08" oy="${s*0.03}"/>
-    </link>
-    <!-- Hip pitch: flexion 120 deg (negative) / extension 30 deg (positive) -->
+      <!-- carries the hip pitch actuator, outside the thigh -->
+      <collision>
+        <origin xyz="0 ${s*0.080} 0" rpy="${pi/2} 0 0"/>
+        <geometry><cylinder radius="0.056" length="0.050"/></geometry>
+      </collision>
+      <xacro:solid_box_inertial m="2.9" x="0.12" y="0.10" z="0.11" ox="-0.02" oy="${s*0.07}"/>
+    </link>
+    <!-- Hip pitch: flexion 89 deg (negative) / extension 29 deg (positive). The thigh meets the
+         hip-yaw link at 91.6 deg flexion and the roll actuator / pelvis at 30 deg extension -->
     <joint name="${side}_hip_pitch_joint" type="revolute">
       <parent link="${side}_hip_roll_link"/>
@@ -106,5 +124,5 @@
       <origin xyz="0 0 0" rpy="0 0 0"/>
       <axis xyz="0 1 0"/>
-      <limit lower="-2.09" upper="0.52" effort="250" velocity="8.0"/>
+      <limit lower="-1.55" upper="0.50" effort="250" velocity="8.0"/>
       <dynamics damping="0.5" friction="0.1"/>
     </joint>
@@ -113,7 +131,8 @@
       <collision>
         <origin xyz="0.005 0 ${-thigh_length*0.47}" rpy="0 0 0"/>
-        <geometry><cylinder radius="0.055" length="${thigh_length*0.68}"/></geometry>
-      </collision>
-      <xacro:solid_cyl_inertial m="5.0" r="0.06" h="${thigh_length}" oz="${-thigh_length*0.4}"/>
+        <geometry><cylinder radius="0.050" length="${thigh_length*0.68}"/></geometry>
+      </collision>
+      <!-- structure + knee actuator at the bottom -->
+      <xacro:solid_cyl_inertial m="4.3" r="0.055" h="${thigh_length}" oz="${-thigh_length*0.55}"/>
     </link>
     <!-- Knee: flexion 0..140 deg -->

File: src/my_robot_description/urdf/my_robot.urdf.xacro (robot description, xacro)
@@ -2,5 +2,5 @@
 <robot name="my_robot" xmlns:xacro="http://www.ros.org/wiki/xacro">
     <xacro:include filename="common_properties.xacro" />
-    <!-- lower body: pelvis (base_link) + two 7-DOF legs, then the 3-DOF waist -->
+    <!-- lower body: pelvis (base_link) + two 7-DOF legs, then the rigid torso -->
     <xacro:include filename="legs.xacro" />
     <xacro:include filename="legs_gazebo.xacro" />

File: src/my_robot_description/urdf/torso.xacro (robot description, xacro)
@@ -1,47 +1,27 @@
 <?xml version="1.0"?>
 <!--
-  HRUH waist: 3-DOF lumbar joint between pelvis and chest, like a human spine.
-    waist_yaw   (z): trunk rotation  +-45 deg
-    waist_roll  (x): side bend       +-20 deg
-    waist_pitch (y): flexion 60 deg (positive, leaning forward) / extension 25 deg
+  HRUH torso: rigid. The chest is bolted to the pelvis through a lumbar block
+  (no waist joints). A 3-DOF waist with all axes in one point could not be built
+  (no room for three 150-200 N m actuators), and the walking policy is meant to
+  balance with the legs while the upper body stays still.
 -->
 <robot xmlns:xacro="http://www.ros.org/wiki/xacro">
-  <xacro:property name="waist_z" value="0.09"/>   <!-- waist pivot above the pelvis frame -->
-  <xacro:property name="chest_z" value="0.04"/>   <!-- chest_hruh origin above the waist pivot -->
-  <joint name="waist_yaw_joint" type="revolute">
+  <xacro:property name="waist_z" value="0.09"/>   <!-- lumbar block (torso_link) above the pelvis frame -->
+  <xacro:property name="chest_z" value="0.04"/>   <!-- chest_hruh origin above torso_link -->
+  <joint name="torso_fixed_joint" type="fixed">
     <parent link="pelvis_link"/>
-    <child link="waist_yaw_link"/>
+    <child link="torso_link"/>
     <origin xyz="0 0 ${waist_z}" rpy="0 0 0"/>
-    <axis xyz="0 0 1"/>
-    <limit lower="-0.79" upper="0.79" effort="150" velocity="4.0"/>
-    <dynamics damping="1.0" friction="0.2"/>
   </joint>
-  <link name="waist_yaw_link">
+  <link name="torso_link">
     <visual>
       <geometry><mesh filename="package://my_robot_description/meshes/legs/waist.obj"/></geometry>
     </visual>
-    <xacro:solid_cyl_inertial m="2.0" r="0.07" h="0.09"/>
-  </link>
-  <joint name="waist_roll_joint" type="revolute">
-    <parent link="waist_yaw_link"/>
-    <child link="waist_roll_link"/>
-    <origin xyz="0 0 0" rpy="0 0 0"/>
-    <axis xyz="1 0 0"/>
-    <limit lower="-0.35" upper="0.35" effort="150" velocity="4.0"/>
-    <dynamics damping="1.0" friction="0.2"/>
-  </joint>
-  <link name="waist_roll_link">
-    <xacro:solid_box_inertial m="0.5" x="0.05" y="0.05" z="0.05"/>
-  </link>
-  <joint name="waist_pitch_joint" type="revolute">
-    <parent link="waist_roll_link"/>
-    <child link="torso_link"/>
-    <origin xyz="0 0 0" rpy="0 0 0"/>
-    <axis xyz="0 1 0"/>
-    <limit lower="-0.44" upper="1.05" effort="200" velocity="4.0"/>
-    <dynamics damping="1.0" friction="0.2"/>
-  </joint>
-  <link name="torso_link">
-    <xacro:solid_box_inertial m="0.5" x="0.05" y="0.05" z="0.05"/>
+    <collision>
+      <origin xyz="0 0 0.005" rpy="0 0 0"/>
+      <geometry><box size="0.14 0.19 0.07"/></geometry>
+    </collision>
+    <!-- lumbar housing (electronics) -->
+    <xacro:solid_box_inertial m="3.0" x="0.14" y="0.19" z="0.07"/>
   </link>
 </robot>
