Commit message: commit

File: install/my_robot_description/share/my_robot_description/urdf/lidar_gz.xacro (robot description, xacro)
@@ -25,36 +25,38 @@
   </joint>
   <!-- Gazebo Sim LiDAR sensor -->
-  <gazebo reference="lidar_link">
-    <sensor name="gpu_lidar" type="gpu_lidar">
-      <pose>0 0 0 0 0 0</pose>
-      <topic>/lidar</topic>
-      <update_rate>60</update_rate>
-      <!-- 360° horizontal + a few vertical beams -> 3D point cloud -->
-      <ray>
-        <scan>
-          <horizontal>
-            <samples>1024</samples>
-            <resolution>1</resolution>
-            <min_angle>-3.14159</min_angle>
-            <max_angle> 3.14159</max_angle>
-          </horizontal>
-          <vertical>
-            <samples>1025</samples>
-            <resolution>1</resolution>
-            <min_angle>-3.14159</min_angle>  <!-- -15° -->
-            <max_angle> 3.14159</max_angle>  <!-- +15° -->
-          </vertical>
-        </scan>
-        <range>
-          <min>0.05</min>
-          <max>45.0</max>
-          <resolution>0.01</resolution>
-        </range>
-      </ray>
-      <!-- Frame on messages; optional but nice to be explicit -->
-      <gz_frame_id>lidar_link</gz_frame_id>
-      <always_on>1</always_on>
-      <visualize>true</visualize>
-    </sensor>
-  </gazebo>
+  <xacro:if value="${enable_lidar}">
+    <gazebo reference="lidar_link">
+      <sensor name="gpu_lidar" type="gpu_lidar">
+        <pose>0 0 0 0 0 0</pose>
+        <topic>/lidar</topic>
+        <update_rate>60</update_rate>
+        <!-- 360° horizontal + a few vertical beams -> 3D point cloud -->
+        <ray>
+          <scan>
+            <horizontal>
+              <samples>1024</samples>
+              <resolution>1</resolution>
+              <min_angle>-3.14159</min_angle>
+              <max_angle> 3.14159</max_angle>
+            </horizontal>
+            <vertical>
+              <samples>1025</samples>
+              <resolution>1</resolution>
+              <min_angle>-3.14159</min_angle>  <!-- -15° -->
+              <max_angle> 3.14159</max_angle>  <!-- +15° -->
+            </vertical>
+          </scan>
+          <range>
+            <min>0.05</min>
+            <max>45.0</max>
+            <resolution>0.01</resolution>
+          </range>
+        </ray>
+        <!-- Frame on messages; optional but nice to be explicit -->
+        <gz_frame_id>lidar_link</gz_frame_id>
+        <always_on>1</always_on>
+        <visualize>true</visualize>
+      </sensor>
+    </gazebo>
+  </xacro:if>
 </robot>

File: install/my_robot_description/share/my_robot_description/urdf/mobile_base.xacro (robot description, xacro)
@@ -36,5 +36,5 @@
                 </geometry>
                 <origin xyz="0 0 0" rpy="${pi / 2.0} 0 0" />
-                <material name="grey" />
+                <material name="red" />
             </visual>
             <collision>
@@ -48,41 +48,35 @@
         </link>
     </xacro:macro>
-    <xacro:wheel_link prefix="right" />
-    <xacro:wheel_link prefix="left" />
-    <link name="caster_wheel_link">
-        <visual>
-            <geometry>
-                <sphere radius="${wheel_radius / 2.0}" />
-            </geometry>
-            <origin xyz="0 0 0" rpy="0 0 0" />
-            <material name="grey" />
-        </visual>
-        <collision>
-            <geometry>
-                <sphere radius="${wheel_radius / 2.0}" />
-            </geometry>
-            <origin xyz="0 0 0" rpy="0 0 0" />
-        </collision>
-        <xacro:sphere_inertia m="10" r="${2*wheel_radius / 2.0}"
-                              xyz="0 0 0" rpy="0 0 0" />
-    </link>
+    <xacro:wheel_link prefix="right_back" />
+    <xacro:wheel_link prefix="left_back" />
+    <xacro:wheel_link prefix="right_front" />
+    <xacro:wheel_link prefix="left_front" />
     <link name="base_footprint">
     </link>
-    <joint name="base_right_wheel_joint" type="continuous">
+    <joint name="base_right_back_wheel_joint" type="continuous">
         <parent link="base_link" />
-        <child link="right_wheel_link" />
+        <child link="right_back_wheel_link" />
         <origin xyz="${-base_length / 4.0} ${-(base_width + wheel_length) / 2.0} 0" rpy="0 0 0" />
         <axis xyz="0 1 0" />
     </joint>
-     <joint name="base_left_wheel_joint" type="continuous">
+    <joint name="base_right_front_wheel_joint" type="continuous">
         <parent link="base_link" />
-        <child link="left_wheel_link" />
+        <child link="right_front_wheel_link" />
+        <origin xyz="${(base_length) / 4.0} ${-(base_width + wheel_length) / 2.0} 0" rpy="0 0 0" />
+        <axis xyz="0 1 0" />
+        <mimic joint="base_right_back_wheel_joint" multiplier="1" />
+    </joint>
+     <joint name="base_left_back_wheel_joint" type="continuous">
+        <parent link="base_link" />
+        <child link="left_back_wheel_link" />
         <origin xyz="${-base_length / 4.0} ${(base_width + wheel_length) / 2.0} 0" rpy="0 0 0" />
         <axis xyz="0 1 0" />
     </joint>
-    <joint name="base_caster_wheel_joint" type="fixed">
+    <joint name="base_left_front_wheel_joint" type="continuous">
         <parent link="base_link" />
-        <child link="caster_wheel_link" />
-        <origin xyz="${base_length / 3.0} 0 ${-wheel_radius / 2.0}" rpy="0 0 0" />
+        <child link="left_front_wheel_link" />
+        <origin xyz="${base_length / 4.0} ${(base_width + wheel_length) / 2.0} 0" rpy="0 0 0" />
+        <axis xyz="0 1 0" />
+        <mimic joint="base_left_back_wheel_joint" multiplier="1" />
     </joint>
     <joint name="base_footprint_joint" type="fixed">

File: install/my_robot_description/share/my_robot_description/urdf/mobile_base_gazebo.xacro (robot description, xacro)
@@ -4,14 +4,15 @@
         <material>Gazebo/Blue</material>
     </gazebo>
-    <gazebo reference="right_wheel_link">
-        <material>Gazebo/Grey</material>
+    <gazebo reference="right_back_wheel_link">
+        <material>Gazebo/Red</material>
     </gazebo>
-    <gazebo reference="left_wheel_link">
-        <material>Gazebo/Grey</material>
+    <gazebo reference="left_back_wheel_link">
+        <material>Gazebo/Red</material>
     </gazebo>
-    <gazebo reference="caster_wheel_link">
-        <material>Gazebo/Grey</material>
-        <mu1 value="0.1" />
-        <mu2 value="0.1" />
+    <gazebo reference="right_front_wheel_link">
+        <material>Gazebo/Red</material>
+    </gazebo>
+    <gazebo reference="left_front_wheel_link">
+        <material>Gazebo/Red</material>
     </gazebo>
     <gazebo>
@@ -39,6 +40,8 @@
             filename="gz-sim-diff-drive-system"
             name="gz::sim::systems::DiffDrive">
-            <left_joint>base_left_wheel_joint</left_joint>
-            <right_joint>base_right_wheel_joint</right_joint>
+            <left_joint>base_left_back_wheel_joint</left_joint>
+            <left_joint>base_left_front_wheel_joint</left_joint>
+            <right_joint>base_right_back_wheel_joint</right_joint>
+            <right_joint>base_right_front_wheel_joint</right_joint>
             <wheel_separation>0.45</wheel_separation>
             <wheel_radius>0.1</wheel_radius>
@@ -51,6 +54,8 @@
             filename="gz-sim-joint-state-publisher-system"
             name="gz::sim::systems::JointStatePublisher">
-            <joint_name>base_left_wheel_joint</joint_name>
-            <joint_name>base_right_wheel_joint</joint_name>
+            <joint_name>base_left_back_wheel_joint</joint_name>
+            <joint_name>base_left_front_wheel_joint</joint_name>
+            <joint_name>base_right_back_wheel_joint</joint_name>
+            <joint_name>base_right_front_wheel_joint</joint_name>
         </plugin>
     </gazebo>

File: install/my_robot_description/share/my_robot_description/urdf/my_robot.urdf.xacro (robot description, xacro)
@@ -8,5 +8,8 @@
     <xacro:include filename="hruh.xacro" />
     <xacro:include filename="hruh_gazebo.xacro" />
-    <!-- <xacro:include filename="stereo_camera.xacro" /> -->
+    <xacro:property name="enable_stereo_cameras" value="true"/>
+    <xacro:property name="enable_rgbd_camera" value="true"/>
+    <xacro:property name="enable_lidar" value="true"/>
+    <xacro:include filename="stereo_camera.xacro" />
     <xacro:include filename="rgbd_camera.xacro"/>
     <!-- <xacro:include filename="camera.xacro" /> -->

File: install/my_robot_description/share/my_robot_description/urdf/rgbd_camera.xacro (robot description, xacro)
@@ -40,24 +40,26 @@
   </joint>
   <!-- Gazebo Sim RGB-D sensor -->
-  <gazebo reference="rgbd_link">
-    <sensor name="rgbd_camera" type="rgbd_camera">
-      <always_on>1</always_on>
-      <update_rate>50</update_rate>
-      <!-- This base topic becomes /camera/image and /camera/depth_image in Gz -->
-      <topic>/camera</topic>
-      <camera>
-        <horizontal_fov>${rgbd_fov}</horizontal_fov>
-        <image>
-          <width>${rgbd_w}</width>
-          <height>${rgbd_h}</height>
-          <format>R8G8B8</format>
-        </image>
-        <clip><near>${rgbd_near}</near><far>${rgbd_far}</far></clip>
-        <!-- Frame id used by the bridges -->
-        <optical_frame_id>rgbd_link</optical_frame_id>
-        <gz_frame_id>rgbd_link</gz_frame_id>
-      </camera>
-      <visualize>true</visualize>
-    </sensor>
-  </gazebo>
+    <xacro:if value="${enable_rgbd_camera}">
+      <gazebo reference="rgbd_link">
+        <sensor name="rgbd_camera" type="rgbd_camera">
+          <always_on>1</always_on>
+          <update_rate>50</update_rate>
+          <!-- This base topic becomes /camera/image and /camera/depth_image in Gz -->
+          <topic>/camera</topic>
+          <camera>
+            <horizontal_fov>${rgbd_fov}</horizontal_fov>
+            <image>
+              <width>${rgbd_w}</width>
+              <height>${rgbd_h}</height>
+              <format>R8G8B8</format>
+            </image>
+            <clip><near>${rgbd_near}</near><far>${rgbd_far}</far></clip>
+            <!-- Frame id used by the bridges -->
+            <optical_frame_id>rgbd_link</optical_frame_id>
+            <gz_frame_id>rgbd_link</gz_frame_id>
+          </camera>
+          <visualize>true</visualize>
+        </sensor>
+      </gazebo>
+    </xacro:if>
 </robot>

File: install/my_robot_description/share/my_robot_description/urdf/stereo_camera.xacro (robot description, xacro)
@@ -34,31 +34,33 @@
   </joint>
   <!-- Cameras for gz (Ionic) -->
-  <gazebo reference="stereo_left">
-    <sensor type="camera" name="left">
-      <always_on>true</always_on>
-      <update_rate>60</update_rate>
-      <gz_frame_id>stereo_left_optical</gz_frame_id>
-      <topic>/stereo/left/image_raw</topic>
-      <camera_info_topic>/stereo/left/camera_info</camera_info_topic>
-      <camera>
-        <horizontal_fov>${fov}</horizontal_fov>
-        <image><width>${cam_w}</width><height>${cam_h}</height><format>R8G8B8</format></image>
-        <clip><near>0.3</near><far>20</far></clip>
-      </camera>
-    </sensor>
-  </gazebo>
-  <gazebo reference="stereo_right">
-    <sensor type="camera" name="right">
-      <always_on>true</always_on>
-      <update_rate>60</update_rate>
-      <gz_frame_id>stereo_right_optical</gz_frame_id>
-      <topic>/stereo/right/image_raw</topic>
-      <camera_info_topic>/stereo/right/camera_info</camera_info_topic>
-      <camera>
-        <horizontal_fov>${fov}</horizontal_fov>
-        <image><width>${cam_w}</width><height>${cam_h}</height><format>R8G8B8</format></image>
-        <clip><near>0.3</near><far>20</far></clip>
-      </camera>
-    </sensor>
-  </gazebo>
+  <xacro:if value="${enable_stereo_cameras}">
+    <gazebo reference="stereo_left">
+      <sensor type="camera" name="left">
+        <always_on>true</always_on>
+        <update_rate>60</update_rate>
+        <gz_frame_id>stereo_left_optical</gz_frame_id>
+        <topic>/stereo/left/image_raw</topic>
+        <camera_info_topic>/stereo/left/camera_info</camera_info_topic>
+        <camera>
+          <horizontal_fov>${fov}</horizontal_fov>
+          <image><width>${cam_w}</width><height>${cam_h}</height><format>R8G8B8</format></image>
+          <clip><near>0.3</near><far>20</far></clip>
+        </camera>
+      </sensor>
+    </gazebo>
+    <gazebo reference="stereo_right">
+      <sensor type="camera" name="right">
+        <always_on>true</always_on>
+        <update_rate>60</update_rate>
+        <gz_frame_id>stereo_right_optical</gz_frame_id>
+        <topic>/stereo/right/image_raw</topic>
+        <camera_info_topic>/stereo/right/camera_info</camera_info_topic>
+        <camera>
+          <horizontal_fov>${fov}</horizontal_fov>
+          <image><width>${cam_w}</width><height>${cam_h}</height><format>R8G8B8</format></image>
+          <clip><near>0.3</near><far>20</far></clip>
+        </camera>
+      </sensor>
+    </gazebo>
+  </xacro:if>
 </robot>
